File: 68kt.sch (KiCad schematic (older format))
At the start: 4 parts

Commit message: updates
Parts:
- added C? (x2): 10uF (tantalum), symbol Device:CP
- added C?: 10nF, symbol Device:CP
- added C?: 4.7uF, symbol Device:CP
- added D?: PWR_GREEN, symbol Device:LED
- added FB?: Ferrite_Bead, symbol Device:Ferrite_Bead
- added J?: LOADER_CON, symbol Connector_Generic:Conn_01x03
- added J?: SPI, symbol Connector_Generic:Conn_01x04
- added J?: I2C, symbol Connector_Generic:Conn_01x03
- added J?: 68KT_CON, symbol Connector_Generic:Conn_01x03
- added J?: USB, symbol Connector_Generic:Conn_01x04
- added J?: USB_B_Micro, symbol Connector:USB_B_Micro
- added R?: 82, symbol Device:R
- added U?: AMS1117-3.3, Package_TO_SOT_SMD:SOT-223-3_TabPin2, symbol Regulator_Linear:AMS1117-3.3
Connections:
- net +3V3: now also C?.1, U?.2 (VO)
- net +5V: now also C?.1, C?.1, FB?.2, U?.3 (VI)
- net GND: now also C?.2, C?.2, C?.2, C?.2, D?.1 (K), J?.3 (Pin_3), J?.3 (Pin_3), J?.3 (Pin_3), J?.4 (Pin_4), J?.4 (Pin_4), J?.5 (GND), J?.6 (Shield), U?.1 (GND)
- new net: D?.2 (A), R?.2
- new net 68KT_CON_RX: J?.1 (Pin_1)
- new net 68KT_CON_TX: J?.2 (Pin_2)
- new net LOADER_CON_RX: J?.1 (Pin_1)
- new net LOADER_CON_TX: J?.2 (Pin_2)
- new net MISO: J?.3 (Pin_3)
- new net MOSI: J?.2 (Pin_2)
- new net SCK: J?.1 (Pin_1)
- new net SCL: J?.1 (Pin_1)
- new net SDA: J?.2 (Pin_2)
- new net USB_D+: J?.2 (Pin_2), J?.3 (D+)
- new net USB_D-: J?.2 (D-), J?.3 (Pin_3)
- new net USB_VBUS: C?.1, FB?.1, J?.1 (Pin_1), J?.1 (VBUS), R?.1
- no-connect marks 0 -> 1
Other:
- note added: "https://www.amazon.co.uk/YOUMILE-Connector-Adapter-2-54mm-Converter-Microusb/dp/B07TVHR9LF\nhttps://datasheet.lcsc.com/szlcsc/1811201117_Advanced-Monolithic-Systems-AMS-AMS1117-3-3_C6186.pdf"
- moved on the sheet: H1, H2, H3, H4

Commit message: updates
Other:
- note added: "JLCPCB Part Reference\n\n74HC04D,653 Hex inverter\n74HC14D,653 Hex inverting Schmitt trigger \n74HC138D,653 3-to-8 line decoder/demultiplexer; inverting\n74HC164D,653 8-bit serial-in, parallel-out shift register\n74HC165D,653 8-bit parallel-in/serial out shift register\n74HC245D,653 Octal bus tranceiver; 3-state\n74HC595D,118 8-bit serial-in, serial or parallel-out shift register with output latc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"
- note added: "Memory Map\n$000000 $0FFFFF 1MiB RAM\n$100000 $17FFFF 1MiB Pseudo ROM\n$180000 $1FFFFF INVALID\n$200000 $27FFFF 1MiB Pseudo IO\n$280000 $3FFFFF INVALID\n$400000 $7FFFFF UNMAPPED\n\nRAM A20 address A19-A1\nROM A21 address A19-A1\nIO A23 address A19-A1\nLOADER (A23-A1)\n\n"
- note added: "TODO\nhalt led\nreset led\n68k clock\natmega clock caps\n68k addressing, /as /dtack, /uds /lds\ncalculate pull pu and pull down resitors\ncheck no shorts\ncheck directions of signals\n\nhttps://www.nxp.com/docs/en/user-guide/MC68332UM.pdf"
- note removed: "JLCPCB Part Reference\n\n74HC00D,653 Quad 2-input NAND gate\n74HC138D,653 3-to-8 line decoder/demultiplexer; inverting\n74HC165D,653 8-bit parallel-in/serial out shift register\n74HC245D,653 Octal bus tranceiver; 3-state\n74HC595D,118 8-bit serial-in, serial or parallel-out shift register with output latches; 3-state\n74HCT04 Hex inverter\n74HCT14 Hex inverting Schmitt trigger \n\n2N7002 MOSFET N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"
- note removed: "Memory Map\n$000000 $0FFFFF 1MiB RAM\n$100000 $17FFFF 1MiB Pseudo ROM\n$180000 $1FFFFF INVALID\n$200000 $27FFFF 1MiB Pseudo IO\n$280000 $3FFFFF INVALID\n$400000 $7FFFFF UNMAPPED\n\nRAM A20 address A19-A1\nROM A21 address A19-A1\nIO A23 address A19-A1\nLOADER (A1-A23)\n\n"
- note removed: "TODO\nhalt led\nreset led\n68k clock\n68k addressing, /as /dtack, /uds /lds\n\nhttps://www.nxp.com/docs/en/user-guide/MC68332UM.pdf"
- moved on the sheet: J?

Commit message: update usb protection
Parts:
- added U?: SRV05-4, Package_TO_SOT_SMD:SOT-23-6, symbol Power_Protection:SRV05-4
Connections:
- net GND: now also U?.2 (VN)
- net USB_D+: now also U?.1 (IO1)
- net USB_D-: now also U?.3 (IO2)
- net USB_VBUS: now also U?.5 (VP)
- no-connect marks 1 -> 3
Other:
- note added: "https://www.amazon.co.uk/YOUMILE-Connector-Adapter-2-54mm-Converter-Microusb/dp/B07TVHR9LF\nhttps://datasheet.lcsc.com/szlcsc/ProTek-Devices-SRV05-4-P-T7_C85364.pdf\nhttps://datasheet.lcsc.com/szlcsc/1811201117_Advanced-Monolithic-Systems-AMS-AMS1117-3-3_C6186.pdf"
- note removed: "https://www.amazon.co.uk/YOUMILE-Connector-Adapter-2-54mm-Converter-Microusb/dp/B07TVHR9LF\nhttps://datasheet.lcsc.com/szlcsc/1811201117_Advanced-Monolithic-Systems-AMS-AMS1117-3-3_C6186.pdf"
Changed lines of the file:
@@
 Memory Map\n$000000 $0FFFFF 1MiB RAM\n$100000 $17FFFF 1MiB Pseudo ROM\n$180000 $1FFFFF INVALID\n$200000 $27FFFF 1MiB Pseudo IO\n$280000 $3FFFFF INVALID\n$400000 $7FFFFF UNMAPPED\n\nRAM A20 address A19-A1\nROM A21 address A19-A1\nIO  A23 address A19-A1\nLOADER (A23-A1)\n\n
 Text Notes 650  5100 0    50   ~ 0
-JLCPCB Part Reference\n\n74HC04D,653 Hex inverter\n74HC14D,653 Hex inverting Schmitt trigger \n74HC138D,653 3-to-8 line decoder/demultiplexer; inverting\n74HC164D,653 8-bit serial-in, parallel-out shift register\n74HC165D,653 8-bit parallel-in/serial out shift register\n74HC245D,653 Octal bus tranceiver; 3-state\n74HC595D,118 8-bit serial-in, serial or parallel-out shift register with output latches; 3-state\n\n\n2N7002 MOSFET N TRENCH 60V 115MA 2.5V @ 250UA 7.5 \nAMS1117-3.3 1A LOW DROPOUT VOLTAGE REGULATOR\nFT232RL-REEL USB UART I.C.\nATMEGA2560-16AU 8-bit Atmel Microcontroller with 16/32/64KB In-System Programmable Flash\nIS62WV51216BLL-55TLI  512K x 16 LOW VOLTAGE,ULTRA LOW POWER CMOS STATIC RAM\n\nX322516MLB4SI SMD CRYSTAL RESONATORS 16MHZ\n\nTAJA106K016RNJ TANTALUM CAPACITORS 10UF 16V CASE-A_3216\n0603WAF820JT5E CHIP RESISTOR - SURFACE MOUNT 82OHMS ±1% 1/10W 0603 ROHS Basic Part \n0603WAF1500T5E  CHIP RESISTOR - SURFACE MOUNT 150OHMS ±1% 1/10W 060\n\n19-217/GHC-YR1S2/3T LIGHT EMITTING DIODES (LED) GREEN 520~535NM 112~258MCD@20MA TOP VIEW 0603 ROHS Basic Part\nvcc=5; i=20; vf=3.3; (vcc-vf)/(i/1000) = 85 Ohms (0.066W) (82 Ohms  0.1W)\n\nKT-0603R LIGHT EMITTING DIODES (LED) RED 520~625NM 90~100M\nvcc=5; i=20; vf=2.1; (vcc-vf)/(i/1000) = 145 Ohms (0.042) (150 Ohms  0.1W)\n\nhttps://ohmslawcalculator.com/led-resistor-calculator
+JLCPCB Part Reference\n\n74HC04D,653 Hex inverter\n74HC14D,653 Hex inverting Schmitt trigger \n74HC138D,653 3-to-8 line decoder/demultiplexer; inverting\n74HC164D,653 8-bit serial-in, parallel-out shift register\n74HC165D,653 8-bit parallel-in/serial out shift register\n74HC245D,653 Octal bus tranceiver; 3-state\n74HC595D,118 8-bit serial-in, serial or parallel-out shift register with output latches; 3-state\n\n\n2N7002 MOSFET N TRENCH 60V 115MA 2.5V @ 250UA 7.5 \nAMS1117-3.3 1A LOW DROPOUT VOLTAGE REGULATOR\nFT232RL-REEL USB UART I.C.\nATMEGA2560-16AU 8-bit Atmel Microcontroller with 16/32/64KB In-System Programmable Flash\nIS62WV51216BLL-55TLI  512K x 16 LOW VOLTAGE,ULTRA LOW POWER CMOS STATIC RAM\n\nSRV05-4-P-T7  ULTRA LOW CAPACITANCE STEERING DIODE/TVS ARRAY\n\nX322516MLB4SI SMD CRYSTAL RESONATORS 16MHZ\n\nTAJA106K016RNJ TANTALUM CAPACITORS 10UF 16V CASE-A_3216\n0603WAF820JT5E CHIP RESISTOR - SURFACE MOUNT 82OHMS ±1% 1/10W 0603 ROHS Basic Part \n0603WAF1500T5E  CHIP RESISTOR - SURFACE MOUNT 150OHMS ±1% 1/10W 060\n\n19-217/GHC-YR1S2/3T LIGHT EMITTING DIODES (LED) GREEN 520~535NM 112~258MCD@20MA TOP VIEW 0603 ROHS Basic Part\nvcc=5; i=20; vf=3.3; (vcc-vf)/(i/1000) = 85 Ohms (0.066W) (82 Ohms  0.1W)\n\nKT-0603R LIGHT EMITTING DIODES (LED) RED 520~625NM 90~100M\nvcc=5; i=20; vf=2.1; (vcc-vf)/(i/1000) = 145 Ohms (0.042) (150 Ohms  0.1W)\n\nhttps://ohmslawcalculator.com/led-resistor-calculator
 Text Notes 650  6000 0    50   ~ 0
 TODO\nhalt led\nreset led\n68k clock\natmega clock caps\n68k addressing, /as /dtack, /uds /lds\ncalculate pull pu and pull down resitors\ncheck no shorts\ncheck directions of signals\n\nhttps://www.nxp.com/docs/en/user-guide/MC68332UM.pdf
@@
 	8500 5750 8500 5850
 Text Notes 6800 6450 0    50   ~ 0
-https://www.amazon.co.uk/YOUMILE-Connector-Adapter-2-54mm-Converter-Microusb/dp/B07TVHR9LF\nhttps://datasheet.lcsc.com/szlcsc/1811201117_Advanced-Monolithic-Systems-AMS-AMS1117-3-3_C6186.pdf
+https://www.amazon.co.uk/YOUMILE-Connector-Adapter-2-54mm-Converter-Microusb/dp/B07TVHR9LF\nhttps://datasheet.lcsc.com/szlcsc/ProTek-Devices-SRV05-4-P-T7_C85364.pdf\nhttps://datasheet.lcsc.com/szlcsc/1811201117_Advanced-Monolithic-Systems-AMS-AMS1117-3-3_C6186.pdf
 $Comp
 L power:GND #PWR?
@@
 Wire Wire Line
 	7600 3800 7700 3800
+$Comp
+L Power_Protection:SRV05-4 U?
+U 1 1 5F9F1E54
+P 6050 5600
+F 0 "U?" H 6200 6050 50  0000 C CNN
+F 1 "SRV05-4" H 6300 6150 50  0000 C CNN
+F 2 "Package_TO_SOT_SMD:SOT-23-6" H 6750 5150 50  0001 C CNN
+F 3 "http://www.onsemi.com/pub/Collateral/SRV05-4-D.PDF" H 6050 5600 50  0001 C CNN
+	1    6050 5600
+	1    0    0    -1
+$EndComp
+Text GLabel 5950 5000 0    50   Output ~ 0
+USB_VBUS
+Text GLabel 5550 5500 0    50   BiDi ~ 0
+USB_D+
+Text GLabel 5550 5700 0    50   BiDi ~ 0
+USB_D-
+Text GLabel 5950 6200 0    50   UnSpc ~ 0
+USB_GND
+NoConn ~ 6550 5500
+NoConn ~ 6550 5700
+Wire Wire Line
+	6050 6100 6050 6200
+Wire Wire Line
+	6050 6200 5950 6200
+Wire Wire Line
+	5950 5000 6050 5000
+Wire Wire Line
+	6050 5000 6050 5100
 $EndSCHEMATC

Commit message: updates
Parts:
- removed C? (x2): 10uF (tantalum), symbol Device:CP
- removed C?: 10nF, symbol Device:CP
- removed C?: 4.7uF, symbol Device:CP
- removed D?: PWR_GREEN, symbol Device:LED
- removed FB?: Ferrite_Bead, symbol Device:Ferrite_Bead
- removed J?: LOADER_CON, symbol Connector_Generic:Conn_01x03
- removed J?: SPI, symbol Connector_Generic:Conn_01x04
- removed J?: I2C, symbol Connector_Generic:Conn_01x03
- removed J?: 68KT_CON, symbol Connector_Generic:Conn_01x03
- removed J?: USB, symbol Connector_Generic:Conn_01x04
- removed J?: USB_B_Micro, symbol Connector:USB_B_Micro
- removed R?: 82, symbol Device:R
- removed U?: SRV05-4, Package_TO_SOT_SMD:SOT-23-6, symbol Power_Protection:SRV05-4
- removed U?: AMS1117-3.3, Package_TO_SOT_SMD:SOT-223-3_TabPin2, symbol Regulator_Linear:AMS1117-3.3
- added J1: USB_B_Micro, 68kt:USB, symbol Connector:USB_B_Micro
- added J2: Conn_02x06_Odd_Even, Connector_PinHeader_2.54mm:PinHeader_2x06_P2.54mm_Vertical, symbol Connector_Generic:Conn_02x06_Odd_Even
- added TP1: Test USB_VBUS, TestPoint:TestPoint_Pad_D1.0mm, symbol Connector:TestPoint
- added TP2: Test USB_D+, TestPoint:TestPoint_Pad_D1.0mm, symbol Connector:TestPoint
- added TP3: Test USB_D-, TestPoint:TestPoint_Pad_D1.0mm, symbol Connector:TestPoint
- added TP4: Test USB_GND, TestPoint:TestPoint_Pad_D1.0mm, symbol Connector:TestPoint
- H1, H2, H3, H4: footprint (none) -> MountingHole:MountingHole_2.2mm_M2_Pad
Connections:
- net 68KT_CON_RX: now also J2.2 (Pin_2)
- net 68KT_CON_TX: now also J2.4 (Pin_4)
- net GND: now also J2.10 (Pin_10), J2.11 (Pin_11), J2.12 (Pin_12)
- net LOADER_CON_RX: now also J2.1 (Pin_1)
- net LOADER_CON_TX: now also J2.3 (Pin_3)
- net MISO: now also J2.9 (Pin_9)
- net MOSI: now also J2.7 (Pin_7)
- net SCK: now also J2.5 (Pin_5)
- net SCL: now also J2.6 (Pin_6)
- net SDA: now also J2.8 (Pin_8)
- net USB_D+: now also J1.3 (D+), TP2.1
- net USB_D-: now also J1.2 (D-), TP3.1
- net USB_VBUS: now also J1.1 (VBUS), TP1.1
- new net USB_GND: J1.5 (GND), J1.6 (Shield), TP4.1
- no-connect marks 3 -> 1
Other:
- note added: "CPU M68000\nCPU clock\nCPU reset\nCPU reset/halt LEDs"
- note added: "External connections and headers"
- note added: "Loader ATmega2560\nLoader reset\nLoader clock\nUSB to serial\nSerial LEDs\nGPIO LEDs"
- note added: "Static RAM\n5V to 3.3 level converters\n\nMemory Map\n$000000 $0FFFFF 1MiB RAM\n$100000 $17FFFF 1MiB Pseudo ROM\n$180000 $1FFFFF INVALID\n$200000 $27FFFF 1MiB Pseudo IO\n$280000 $3FFFFF INVALID\n$400000 $7FFFFF UNMAPPED\n\nRAM A20 address A19-A1\nROM A21 address A19-A1\nIO A23 address A19-A1\nLOADER (A23-A1)"
- note added: "TODO\nhalt led\nreset led\n68k clock\natmega clock caps\n68k addressing, /as /dtack, /uds /lds\ncalculate pull pu and pull down resitors\ncheck no shorts\ncheck directions of signals\n\nchange reset sw to shmit"
- note added: "Transient Voltage Suppressor\nUSB capacitor and ferrite\nPower LED\n3 volt regulator"
- note added: "URLS\nhttps://jlcpcb.com/parts\nhttps://hackaday.com/2016/12/05/taking-it-to-another-level-making-3-3v-and-5v-logic-communicate-with-level-shifters/\nhttps://electronics.stackexchange.com/questions/81580/step-up-3-3v-to-5v-for-digital-i-o\nhttps://electronics.stackexchange.com/questions/476140/driving-a-74hc245-in-one-direction-with-3-3v-when-vcc-is-5v\nhttps://www.eejournal.com/article/ultimate-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"
- note added: "https://www.amazon.co.uk/YOUMILE-Connector-Adapter-2-54mm-Converter-Microusb/dp/B07TVHR9LF"
- note removed: "Memory Map\n$000000 $0FFFFF 1MiB RAM\n$100000 $17FFFF 1MiB Pseudo ROM\n$180000 $1FFFFF INVALID\n$200000 $27FFFF 1MiB Pseudo IO\n$280000 $3FFFFF INVALID\n$400000 $7FFFFF UNMAPPED\n\nRAM A20 address A19-A1\nROM A21 address A19-A1\nIO A23 address A19-A1\nLOADER (A23-A1)\n\n"
- note removed: "Pseudo IO Memory Map\n$200001 CONSOLERX (A1)\n$200002 CONSOLETX (A2)\n$200004 LED0 (A3)\n$200008 LED1 (A4)\n$200010 LED2 (A5)\n$200020 LED3 (A6)\n$200040 LED4 (A7)\n$200080 LED5 (A8)\n$200100 LED6 (A9)\n$200200 LED7 (A10)\n$200400 RTCRX (A11)\n$200800 RTCTX (A12)\n$201000 FUTURE (A13)\n$202000 FUTURE (A14)\n$204000 FUTURE (A15)\n$208000 FUTURE (A16)\n$210000 FUTURE (A17)\n$220000 FUTURE (A18)\n$2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"
- note removed: "TODO\nhalt led\nreset led\n68k clock\natmega clock caps\n68k addressing, /as /dtack, /uds /lds\ncalculate pull pu and pull down resitors\ncheck no shorts\ncheck directions of signals\n\nhttps://www.nxp.com/docs/en/user-guide/MC68332UM.pdf"
- note removed: "URLS\n\nhttps://jlcpcb.com/parts\nhttps://hackaday.com/2016/12/05/taking-it-to-another-level-making-3-3v-and-5v-logic-communicate-with-level-shifters/\nhttps://electronics.stackexchange.com/questions/81580/step-up-3-3v-to-5v-for-digital-i-o\nhttps://electronics.stackexchange.com/questions/476140/driving-a-74hc245-in-one-direction-with-3-3v-when-vcc-is-5v\nhttps://www.eejournal.com/article/ultimat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"
- note removed: "https://www.amazon.co.uk/YOUMILE-Connector-Adapter-2-54mm-Converter-Microusb/dp/B07TVHR9LF\nhttps://datasheet.lcsc.com/szlcsc/ProTek-Devices-SRV05-4-P-T7_C85364.pdf\nhttps://datasheet.lcsc.com/szlcsc/1811201117_Advanced-Monolithic-Systems-AMS-AMS1117-3-3_C6186.pdf"
- moved on the sheet: H1, H2, H3, H4

Commit message: updates
Parts:
- removed J2: Conn_02x06_Odd_Even, Connector_PinHeader_2.54mm:PinHeader_2x06_P2.54mm_Vertical, symbol Connector_Generic:Conn_02x06_Odd_Even
- removed TP1: Test USB_VBUS, TestPoint:TestPoint_Pad_D1.0mm, symbol Connector:TestPoint
- removed TP2: Test USB_D+, TestPoint:TestPoint_Pad_D1.0mm, symbol Connector:TestPoint
- removed TP3: Test USB_D-, TestPoint:TestPoint_Pad_D1.0mm, symbol Connector:TestPoint
- removed TP4: Test USB_GND, TestPoint:TestPoint_Pad_D1.0mm, symbol Connector:TestPoint
- added J2: I2C, Connector_PinHeader_2.54mm:PinHeader_1x04_P2.54mm_Vertical, symbol Connector_Generic:Conn_01x04
- added J3: Consoles, Connector_PinHeader_2.54mm:PinHeader_2x06_P2.54mm_Vertical, symbol Connector_Generic:Conn_02x06_Odd_Even
- added J4: SPI, Connector_PinHeader_2.54mm:PinHeader_2x03_P2.54mm_Vertical, symbol Connector_Generic:Conn_02x03_Odd_Even
- added JP1: Jumper_2_Open, Connector_PinHeader_2.54mm:PinHeader_1x02_P2.54mm_Vertical, symbol Jumper:Jumper_2_Open
Connections:
- net +5V: now also JP1.2 (B)
- net 68KT_CON_RX: now also J3.8 (Pin_8)
- net 68KT_CON_TX: now also J3.10 (Pin_10)
- net GND: now also J2.1 (Pin_1), J3.1 (Pin_1), J3.2 (Pin_2), J4.6 (Pin_6)
- net LOADER_CON_RX: now also J3.7 (Pin_7)
- net LOADER_CON_TX: now also J3.9 (Pin_9)
- net MISO: now also J4.1 (Pin_1)
- net MOSI: now also J4.4 (Pin_4)
- net SCK: now also J4.3 (Pin_3)
- net SCL: now also J2.3 (Pin_3)
- net SDA: now also J2.2 (Pin_2)
- new net +5V_JMP: J2.4 (Pin_4), J3.5 (Pin_5), J3.6 (Pin_6), J4.2 (Pin_2), JP1.1 (A)
- new net ~LOADER_RESET: J4.5 (Pin_5)
- no-connect marks 1 -> 5
Other:
- moved on the sheet: J1
