File: CPU.sch (KiCad schematic (older format))
At the start: 10 parts, among them SW2 SW_RESET, U5 68000D, Y2 16MHz

Commit message: updates
Parts:
- removed C15: 22nF, symbol Device:C
- removed Y2: 16MHz, symbol Device:Crystal_GND24
- added C? (x2): 22nF, symbol Device:C
- added R? (x2): R, symbol Device:R
- added U?: 74LS138, symbol 74xx:74LS138
- added U?: 74HC164, symbol 74xx:74HC164
- added U?: 74HCT04, symbol 74xx:74HCT04
- added U? (x7): 74HC04, symbol 74xx:74HC04
- added Y?: 16MHz, symbol Device:Crystal_GND24
Connections:
- net +5V: now also U?.1 (DSA), U?.14 (VCC), U?.16 (VCC), U?.2 (DSB)
- net AS: now also U?.1
- net CLOCK: now also U?.4, U?.8 (CP)
- net GND: now also C?.1, C?.1, U?.7 (GND), U?.8 (GND)
- net ~DTACK: now also U?.10 (Q4)
- net ~BERR: now reaches U5.22 (BERR)
- net ~BERR: now also U?.13 (Q7)
- new net: U?.2, U?.9 (~MR)
- new net: C?.2, R?.2, U?.1, Y?.1
- new net: C?.2, R?.2, Y?.3
- new net: R?.1, R?.1, U?.2, U?.3
Other:
- note added: "Level of drive: 10uW\nEquivalent Series Resistance(ESR) @16MHz: 60-80 ΩMax\nCl (asked on twitter): ? pF\nCo: 7pF\n\nhttps://www.st.com/content/ccc/resource/technical/document/application_note/c6/eb/5e/11/e3/69/43/eb/CD00221665.pdf/files/CD00221665.pdf/jcr:content/translations/en.CD00221665.pdf\nhttp://ww1.microchip.com/downloads/en/appnotes/00826a.pdf\nhttps://www.electronics-tutorials.ws/oscilla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"

Commit message: updates
Parts:
- removed U?: 74LS138, symbol 74xx:74LS138
- removed U?: 74HCT04, symbol 74xx:74HCT04
- added C? (x2): 22nF, symbol Device:C
- added D13: HALT_LED_RED, LED_SMD:LED_0603_1608Metric, symbol Device:LED
- added D14: RESET_LED_RED, LED_SMD:LED_0603_1608Metric, symbol Device:LED
- added R25, R28: 150, Resistor_SMD:R_0603_1608Metric, symbol Device:R
- added R29: 4.7k, symbol Device:R
- added R? (x3): R, symbol Device:R
- added U? (x2): 74HC04, Package_SO:SOIC-14_3.9x8.7mm_P1.27mm, symbol 74xx:74HC04
- added Y?: 8Mhz, Crystal:Crystal_SMD_5032-4Pin_5.0x3.2mm, symbol Device:Crystal_GND24
- C20: renamed from C13; footprint (none) -> Capacitor_SMD:C_0603_1608Metric; JLPCB Datasheet (none) -> https://datasheet.lcsc.com/szlcsc/YAGEO-CC0603KRX7R9BB104_C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; JLPCB Part (none) -> CC0603KRX7R9BB104
- C21: renamed from C14; footprint (none) -> Capacitor_SMD:C_0603_1608Metric; JLPCB Datasheet (none) -> https://datasheet.lcsc.com/szlcsc/YAGEO-CC0603KRX7R9BB104_C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; JLPCB Part (none) -> CC0603KRX7R9BB104
- C24: renamed from C16; footprint (none) -> Capacitor_SMD:C_0603_1608Metric; JLPCB Datasheet (none) -> https://datasheet.lcsc.com/szlcsc/YAGEO-CC0603KRX7R9BB104_C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; JLPCB Part (none) -> CC0603KRX7R9BB104
- U10: renamed from U5; footprint (none) -> Package_DIP:DIP-64_W25.4mm_Socket
- U11: renamed from U?; footprint (none) -> Package_SO:SOIC-14_3.9x8.7mm_P1.27mm; JLPCB Datasheet (none) -> https://datasheet.lcsc.com/szlcsc/Nexperia-74HC04D-653_C559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; JLPCB Part (none) -> 74HC04D,653
- U12: renamed from U?; footprint (none) -> Package_SO:SOIC-14_3.9x8.7mm_P1.27mm; JLPCB Datasheet (none) -> 74HC164D,653; JLPCB Part (none) -> 74HC164D,653
- Y2: renamed from Y?; value 16MHz -> 8Mhz; footprint (none) -> Crystal:Crystal_SMD_5032-4Pin_5.0x3.2mm; JLPCB Datasheet (none) -> https://datasheet.lcsc.com/szlcsc/1903061615_Yangxing-Tech-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; JLPCB Part (none) -> X50328MSB2GI
- gave numbers to parts that had none: 4
- renumbered D13 to D12, R96 to R26, R97 to R27
Connections:
- net +5V: now also U11.14 (VCC)
- net AS: now also U11.11
- net CLOCK: now also U?.4
- net GND: now also U11.13, U11.7 (GND), C?.1, C?.1, R25.2, R28.2, Y?.2, Y?.4
- net ~RESET: now also U11.9
- net at U11.8: now also D14.2 (A)
- net BG: now reaches U10.11 (BG)
- net BGACK: now reaches U10.12 (BGACK)
- net BR: now reaches U10.13 (BR)
- net VMA: now reaches U10.19 (VMA)
- net E: now reaches U10.20 (E)
- net VPA: now reaches U10.21 (VPA)
- net IPL2: now reaches U10.23 (IPL2)
- net IPL1: now reaches U10.24 (IPL1)
- net IPL0: now reaches U10.25 (IPL0)
- net FC2: now reaches U10.26 (FC2)
- net FC1: now reaches U10.27 (FC1)
- net FC0: now reaches U10.28 (FC0)
- new net: D13.1 (K), R25.1
- new net: D14.1 (K), R28.1
- new net: C?.2, R?.1, U?.1, Y?.1
- new net: C?.2, R?.2, Y?.3
- new net: R?.1, R?.2, U?.2, U?.3
- no-connect marks 0 -> 1
Other:
- note added: "KT-0603R LIGHT EMITTING DIODES (LED) RED 520~625NM 90~100M\n0603WAF1500T5E CHIP RESISTOR - SURFACE MOUNT 150OHMS ±1% 1/10W 0603 ROHS\n\nvcc=5; i=20; vf=2; (vcc-vf)/(i/1000); (i/1000)*(vcc-vf) = 150 Ohms, .06 W\nBest match is 150 Ohms 1/10thW (0.1W) resister"
- moved on the sheet: C20, C21, C22, C23, C24, D12, R23, R24, R26, R27, SW2, U10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

Commit message: updates
Parts:
- removed C23: 22nF, symbol Device:C
- removed C24: 100nF, Capacitor_SMD:C_0603_1608Metric, symbol Device:C
- removed R23, R?: R, symbol Device:R
- removed unit 1 of U11
- removed unit 2 of U11
- removed Y2: 8Mhz, Crystal:Crystal_SMD_5032-4Pin_5.0x3.2mm, symbol Device:Crystal_GND24
- added JP2: SolderJumper_WS1, Jumper:SolderJumper-2_P1.3mm_Open_Pad1.0x1.5mm, symbol Jumper:SolderJumper_2_Open
- added JP3: SolderJumper_WS4, Jumper:SolderJumper-2_P1.3mm_Open_Pad1.0x1.5mm, symbol Jumper:SolderJumper_2_Open
- added JP4: SolderJumper_WS7, Jumper:SolderJumper-2_P1.3mm_Open_Pad1.0x1.5mm, symbol Jumper:SolderJumper_2_Open
- added JP5: SolderJumper_WS9, Jumper:SolderJumper-2_P1.3mm_Open_Pad1.0x1.5mm, symbol Jumper:SolderJumper_2_Open
- added JP6: SolderJumper_WS12, Jumper:SolderJumper-2_P1.3mm_Open_Pad1.0x1.5mm, symbol Jumper:SolderJumper_2_Open
- added R25, R28, R29, R31, R32, R33, R34, R35, R36, R37: 4.7k, symbol Device:R
- added R30: R, symbol Device:R
- added U12: 74HC14, Package_SO:SOIC-14_3.9x8.7mm_P1.27mm, symbol 74xx:74HC14
- added U14: 74HC164, Package_SO:SOIC-14_3.9x8.7mm_P1.27mm, symbol 74xx:74HC164
- C22: value 22nF -> F; footprint (none) -> Capacitor_SMD:C_0603_1608Metric; JLPCB Datasheet (none) -> https://datasheet.lcsc.com/szlcsc/YAGEO-CC0603KRX7R9BB104_C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; JLPCB Part (none) -> CC0603KRX7R9BB104
- D12: footprint (none) -> Diode_SMD:D_SMA; JLPCB Datasheet (none) -> https://datasheet.lcsc.com/szlcsc/MDD-Jiangsu-Yutai-Elec-M7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; JLPCB Part (none) -> M7
- R24: value R -> 4.7k
- R27: value 330 -> 4.7k
- U10: JLPCB Datasheet (none) -> N/A; JLPCB Part (none) -> N/A
- U13: renamed from U12; JLPCB Datasheet 74HC164D,653 -> https://datasheet.lcsc.com/szlcsc/Nexperia-74HC164D-653_C68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; JLPCB Part 74HC164D,653 -> 74HC164D,653
- gave numbers to parts that had none: 6
- renumbered R29 to R23, R25 to R38, R28 to R41
Connections:
- net +5V: now also R23.1, R24.1, R27.1, R25.1, R28.1, R29.1, R31.1, R32.1, R33.1, R34.1, R35.1, R36.1, R37.1, U12.14 (VCC), U14.14 (VCC); no longer D12.1 (K), U13.1 (DSA), U13.2 (DSB)
- net AS: now also U11.13
- net BG: now also R27.2
- net BGACK: now also R26.2
- net BR: now also R28.2
- net CLOCK: now also U14.8 (CP)
- net E: now also R35.2
- net FC0: now also R31.2
- net FC1: now also R32.2
- net FC2: now also R33.2
- net GND: now also C22.2, SW2.1, U12.11, U12.13, U12.7 (GND), U14.7 (GND); no longer C22.1, R27.2, U11.13
- net IPL0: now also R23.2
- net IPL1: now also R24.2
- net IPL2: now also R25.2
- net VMA: now also R34.2
- net VPA: now also R36.2
- net ~BERR: now also U14.13 (Q7); no longer U13.13 (Q7)
- net ~DTACK: now also JP2.2 (B), JP3.2 (B), JP4.2 (B), JP5.2 (B), JP6.2 (B), U14.12 (Q6); no longer U13.10 (Q4)
- net ~HALT: now also U11.5, U12.8
- net ~RESET: now also U12.4; no longer D12.2 (A), R26.2, SW2.1
- net at U13.12 (Q6): now also JP4.1 (A)
- net at U13.3 (Q0): now also JP2.1 (A)
- net at U13.6 (Q3): now also JP3.1 (A)
- net at U13.9 (~MR): now also U11.10
- net at U11.6: now also D13.2 (A)
- net at U11.12: now also U14.9 (~MR)
- net at SW2.2: now also D12.2 (A), R29.2, R30.1; no longer R27.1
- new net: R37.2, U13.1 (DSA), U13.2 (DSB)
- new net: U13.13 (Q7), U14.1 (DSA), U14.2 (DSB)
- new net: C22.1, D12.1 (K), R30.2, U12.1, U12.5
- new net: U12.2, U12.3
- new net: U12.6, U12.9
- new net: JP6.1 (A), U14.10 (Q4)
- new net: JP5.1 (A), U14.4 (Q1)
- no-connect marks 1 -> 10
Other:
- note added: "KT-0603R LIGHT EMITTING DIODES (LED) RED 520~~625NM 90~~100M\n0603WAF1500T5E CHIP RESISTOR - SURFACE MOUNT 150OHMS ±1% 1/10W 0603 ROHS\n\nvcc=5; i=20; vf=2; (vcc-vf)/(i/1000); (i/1000)*(vcc-vf) = 150 Ohms, .06 W\nBest match is 150 Ohms 1/10thW (0.1W) resister"
- note added: "Level of drive: 10uW, Equivalent Series Resistance(ESR) @16MHz: 60-80 ΩMax, Cl (asked on twitter): ? pF, Co: 7pF\nhttps://www.st.com/content/ccc/resource/technical/document/application_note/c6/eb/5e/11/e3/\n69/43/eb/CD00221665.pdf/files/CD00221665.pdf/jcr:content/translations/en.CD00221665.pdf\nhttp://ww1.microchip.com/downloads/en/appnotes/00826a.pdf\nhttps://www.electronics-tutorials.ws/oscilla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"
- note added: "http://www.labbookpages.co.uk/electronics/debounce.html\nhttp://wilsonminesco.com/6502primer/RSTreqs.html"
- note removed: "KT-0603R LIGHT EMITTING DIODES (LED) RED 520~625NM 90~100M\n0603WAF1500T5E CHIP RESISTOR - SURFACE MOUNT 150OHMS ±1% 1/10W 0603 ROHS\n\nvcc=5; i=20; vf=2; (vcc-vf)/(i/1000); (i/1000)*(vcc-vf) = 150 Ohms, .06 W\nBest match is 150 Ohms 1/10thW (0.1W) resister"
- note removed: "Level of drive: 10uW\nEquivalent Series Resistance(ESR) @16MHz: 60-80 ΩMax\nCl (asked on twitter): ? pF\nCo: 7pF\n\nhttps://www.st.com/content/ccc/resource/technical/document/application_note/c6/eb/5e/11/e3/69/43/eb/CD00221665.pdf/files/CD00221665.pdf/jcr:content/translations/en.CD00221665.pdf\nhttp://ww1.microchip.com/downloads/en/appnotes/00826a.pdf\nhttps://www.electronics-tutorials.ws/oscilla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"
- moved on the sheet: C20, C21, C23, C24, D13, D14, R23, R38, R39, R40, R41, U11A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

Commit message: update
Parts:
- C23, C24: footprint (none) -> Capacitor_SMD:C_0603_1608Metric
- R23, R24, R25, R26, R27, R28, R29, R31, R32, R33, R34, R35, R36, R37: footprint (none) -> Resistor_SMD:R_0603_1608Metric; JLPCB Datasheet (none) -> https://datasheet.lcsc.com/szlcsc/Uniroyal-Elec-0603WAF4701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; JLPCB Part (none) -> 0603WAF4701T5E
- R30, R39, R40: footprint (none) -> Resistor_SMD:R_0603_1608Metric
- SW2: footprint (none) -> Button_Switch_SMD:SW_Push_1P1T_NO_6x6mm_H9.5mm; JLPCB Datasheet (none) -> https://datasheet.lcsc.com/szlcsc/2006230332_USAKRO-UK-B022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; JLPCB Part (none) -> UK-B0228-G5-160-JZ
Changed lines of the file:
@@
 F 0 "R23" H 3870 4246 50  0000 L CNN
 F 1 "4.7k" H 3870 4155 50  0000 L CNN
-F 2 "" V 3730 4200 50  0001 C CNN
+F 2 "Resistor_SMD:R_0603_1608Metric" V 3730 4200 50  0001 C CNN
 F 3 "~" H 3800 4200 50  0001 C CNN
+F 4 "https://datasheet.lcsc.com/szlcsc/Uniroyal-Elec-0603WAF4701T5E_C23162.pdf" H 3800 4200 50  0001 C CNN "JLPCB Datasheet"
+F 5 "0603WAF4701T5E " H 3800 4200 50  0001 C CNN "JLPCB Part"
 	1    3800 4200
 	0    1    1    0
@@
 F 0 "C23" V 8100 2700 50  0000 R CNN
 F 1 "22nF" V 8200 2700 50  0000 R CNN
-F 2 "" H 8188 2600 50  0001 C CNN
+F 2 "Capacitor_SMD:C_0603_1608Metric" H 8188 2600 50  0001 C CNN
 F 3 "~" H 8150 2750 50  0001 C CNN
 	1    8150 2750
@@
 F 0 "C24" V 8100 3400 50  0000 R CNN
 F 1 "22nF" V 8200 3400 50  0000 R CNN
-F 2 "" H 8188 3300 50  0001 C CNN
+F 2 "Capacitor_SMD:C_0603_1608Metric" H 8188 3300 50  0001 C CNN
 F 3 "~" H 8150 3450 50  0001 C CNN
 	1    8150 3450
@@
 F 0 "R39" H 9020 3496 50  0000 L CNN
 F 1 "R" H 9020 3405 50  0000 L CNN
-F 2 "" V 8880 3450 50  0001 C CNN
+F 2 "Resistor_SMD:R_0603_1608Metric" V 8880 3450 50  0001 C CNN
 F 3 "~" H 8950 3450 50  0001 C CNN
 	1    8950 3450
@@
 F 0 "R40" H 9320 3096 50  0000 L CNN
 F 1 "R" H 9320 3005 50  0000 L CNN
-F 2 "" V 9180 3050 50  0001 C CNN
+F 2 "Resistor_SMD:R_0603_1608Metric" V 9180 3050 50  0001 C CNN
 F 3 "~" H 9250 3050 50  0001 C CNN
 	1    9250 3050
@@
 F 0 "R29" H 4170 1146 50  0000 L CNN
 F 1 "4.7k" H 4170 1055 50  0000 L CNN
-F 2 "" V 4030 1100 50  0001 C CNN
+F 2 "Resistor_SMD:R_0603_1608Metric" V 4030 1100 50  0001 C CNN
 F 3 "~" H 4100 1100 50  0001 C CNN
+F 4 "https://datasheet.lcsc.com/szlcsc/Uniroyal-Elec-0603WAF4701T5E_C23162.pdf" H 4100 1100 50  0001 C CNN "JLPCB Datasheet"
+F 5 "0603WAF4701T5E " H 4100 1100 50  0001 C CNN "JLPCB Part"
 	1    4100 1100
 	1    0    0    -1
@@
 F 0 "SW2" H 4100 2335 50  0000 C CNN
 F 1 "SW_RESET" H 4100 2244 50  0000 C CNN
-F 2 "" H 4100 2250 50  0001 C CNN
+F 2 "Button_Switch_SMD:SW_Push_1P1T_NO_6x6mm_H9.5mm" H 4100 2250 50  0001 C CNN
 F 3 "~" H 4100 2250 50  0001 C CNN
+F 4 "https://datasheet.lcsc.com/szlcsc/2006230332_USAKRO-UK-B0228-G5-160-JZ_C620316.pdf" H 4100 2050 50  0001 C CNN "JLPCB Datasheet"
+F 5 "UK-B0228-G5-160-JZ " H 4100 2050 50  0001 C CNN "JLPCB Part"
 	1    4100 2050
 	0    -1   -1   0
@@
 F 0 "R30" V 4557 1850 50  0000 C CNN
 F 1 "R" V 4466 1850 50  0000 C CNN
-F 2 "" V 4280 1850 50  0001 C CNN
+F 2 "Resistor_SMD:R_0603_1608Metric" V 4280 1850 50  0001 C CNN
 F 3 "~" H 4350 1850 50  0001 C CNN
 	1    4350 1850
@@
 F 0 "R37" H 5470 5396 50  0000 L CNN
 F 1 "4.7k" H 5470 5305 50  0000 L CNN
-F 2 "" V 5330 5350 50  0001 C CNN
+F 2 "Resistor_SMD:R_0603_1608Metric" V 5330 5350 50  0001 C CNN
 F 3 "~" H 5400 5350 50  0001 C CNN
+F 4 "https://datasheet.lcsc.com/szlcsc/Uniroyal-Elec-0603WAF4701T5E_C23162.pdf" H 5400 5350 50  0001 C CNN "JLPCB Datasheet"
+F 5 "0603WAF4701T5E " H 5400 5350 50  0001 C CNN "JLPCB Part"
 	1    5400 5350
 	1    0    0    -1
@@
 F 0 "R24" H 3870 4546 50  0000 L CNN
 F 1 "4.7k" H 3870 4455 50  0000 L CNN
-F 2 "" V 3730 4500 50  0001 C CNN
+F 2 "Resistor_SMD:R_0603_1608Metric" V 3730 4500 50  0001 C CNN
 F 3 "~" H 3800 4500 50  0001 C CNN
+F 4 "https://datasheet.lcsc.com/szlcsc/Uniroyal-Elec-0603WAF4701T5E_C23162.pdf" H 3800 4500 50  0001 C CNN "JLPCB Datasheet"
+F 5 "0603WAF4701T5E " H 3800 4500 50  0001 C CNN "JLPCB Part"
 	1    3800 4500
 	0    1    1    0
@@
 F 0 "R25" H 3870 4846 50  0000 L CNN
 F 1 "4.7k" H 3870 4755 50  0000 L CNN
-F 2 "" V 3730 4800 50  0001 C CNN
+F 2 "Resistor_SMD:R_0603_1608Metric" V 3730 4800 50  0001 C CNN
 F 3 "~" H 3800 4800 50  0001 C CNN
+F 4 "https://datasheet.lcsc.com/szlcsc/Uniroyal-Elec-0603WAF4701T5E_C23162.pdf" H 3800 4800 50  0001 C CNN "JLPCB Datasheet"
+F 5 "0603WAF4701T5E " H 3800 4800 50  0001 C CNN "JLPCB Part"
 	1    3800 4800
 	0    1    1    0
@@
 F 0 "R26" H 3870 5146 50  0000 L CNN
 F 1 "4.7k" H 3870 5055 50  0000 L CNN
-F 2 "" V 3730 5100 50  0001 C CNN
+F 2 "Resistor_SMD:R_0603_1608Metric" V 3730 5100 50  0001 C CNN
 F 3 "~" H 3800 5100 50  0001 C CNN
+F 4 "https://datasheet.lcsc.com/szlcsc/Uniroyal-Elec-0603WAF4701T5E_C23162.pdf" H 3800 5100 50  0001 C CNN "JLPCB Datasheet"
+F 5 "0603WAF4701T5E " H 3800 5100 50  0001 C CNN "JLPCB Part"
 	1    3800 5100
 	0    1    1    0
@@
 F 0 "R27" H 3870 5446 50  0000 L CNN
 F 1 "4.7k" H 3870 5355 50  0000 L CNN
-F 2 "" V 3730 5400 50  0001 C CNN
+F 2 "Resistor_SMD:R_0603_1608Metric" V 3730 5400 50  0001 C CNN
 F 3 "~" H 3800 5400 50  0001 C CNN
+F 4 "https://datasheet.lcsc.com/szlcsc/Uniroyal-Elec-0603WAF4701T5E_C23162.pdf" H 3800 5400 50  0001 C CNN "JLPCB Datasheet"
+F 5 "0603WAF4701T5E " H 3800 5400 50  0001 C CNN "JLPCB Part"
 	1    3800 5400
 	0    1    1    0
@@
 F 0 "R28" H 3870 5746 50  0000 L CNN
 F 1 "4.7k" H 3870 5655 50  0000 L CNN
-F 2 "" V 3730 5700 50  0001 C CNN
+F 2 "Resistor_SMD:R_0603_1608Metric" V 3730 5700 50  0001 C CNN
 F 3 "~" H 3800 5700 50  0001 C CNN
+F 4 "https://datasheet.lcsc.com/szlcsc/Uniroyal-Elec-0603WAF4701T5E_C23162.pdf" H 3800 5700 50  0001 C CNN "JLPCB Datasheet"
+F 5 "0603WAF4701T5E " H 3800 5700 50  0001 C CNN "JLPCB Part"
 	1    3800 5700
 	0    1    1    0
@@
 F 0 "R31" H 4670 4246 50  0000 L CNN
 F 1 "4.7k" H 4670 4155 50  0000 L CNN
-F 2 "" V 4530 4200 50  0001 C CNN
+F 2 "Resistor_SMD:R_0603_1608Metric" V 4530 4200 50  0001 C CNN
 F 3 "~" H 4600 4200 50  0001 C CNN
+F 4 "https://datasheet.lcsc.com/szlcsc/Uniroyal-Elec-0603WAF4701T5E_C23162.pdf" H 4600 4200 50  0001 C CNN "JLPCB Datasheet"
+F 5 "0603WAF4701T5E " H 4600 4200 50  0001 C CNN "JLPCB Part"
 	1    4600 4200
 	0    1    1    0
@@
 F 0 "R32" H 4670 4546 50  0000 L CNN
 F 1 "4.7k" H 4670 4455 50  0000 L CNN
-F 2 "" V 4530 4500 50  0001 C CNN
+F 2 "Resistor_SMD:R_0603_1608Metric" V 4530 4500 50  0001 C CNN
 F 3 "~" H 4600 4500 50  0001 C CNN
+F 4 "https://datasheet.lcsc.com/szlcsc/Uniroyal-Elec-0603WAF4701T5E_C23162.pdf" H 4600 4500 50  0001 C CNN "JLPCB Datasheet"
+F 5 "0603WAF4701T5E " H 4600 4500 50  0001 C CNN "JLPCB Part"
 	1    4600 4500
 	0    1    1    0
@@
 F 0 "R33" H 4670 4846 50  0000 L CNN
 F 1 "4.7k" H 4670 4755 50  0000 L CNN
-F 2 "" V 4530 4800 50  0001 C CNN
+F 2 "Resistor_SMD:R_0603_1608Metric" V 4530 4800 50  0001 C CNN
 F 3 "~" H 4600 4800 50  0001 C CNN
+F 4 "https://datasheet.lcsc.com/szlcsc/Uniroyal-Elec-0603WAF4701T5E_C23162.pdf" H 4600 4800 50  0001 C CNN "JLPCB Datasheet"
+F 5 "0603WAF4701T5E " H 4600 4800 50  0001 C CNN "JLPCB Part"
 	1    4600 4800
 	0    1    1    0
@@
 F 0 "R34" H 4670 5146 50  0000 L CNN
 F 1 "4.7k" H 4670 5055 50  0000 L CNN
-F 2 "" V 4530 5100 50  0001 C CNN
+F 2 "Resistor_SMD:R_0603_1608Metric" V 4530 5100 50  0001 C CNN
 F 3 "~" H 4600 5100 50  0001 C CNN
+F 4 "https://datasheet.lcsc.com/szlcsc/Uniroyal-Elec-0603WAF4701T5E_C23162.pdf" H 4600 5100 50  0001 C CNN "JLPCB Datasheet"
+F 5 "0603WAF4701T5E " H 4600 5100 50  0001 C CNN "JLPCB Part"
 	1    4600 5100
 	0    1    1    0
@@
 F 0 "R35" H 4670 5446 50  0000 L CNN
 F 1 "4.7k" H 4670 5355 50  0000 L CNN
-F 2 "" V 4530 5400 50  0001 C CNN
+F 2 "Resistor_SMD:R_0603_1608Metric" V 4530 5400 50  0001 C CNN
 F 3 "~" H 4600 5400 50  0001 C CNN
+F 4 "https://datasheet.lcsc.com/szlcsc/Uniroyal-Elec-0603WAF4701T5E_C23162.pdf" H 4600 5400 50  0001 C CNN "JLPCB Datasheet"
+F 5 "0603WAF4701T5E " H 4600 5400 50  0001 C CNN "JLPCB Part"
 	1    4600 5400
 	0    1    1    0
@@
 F 0 "R36" H 4670 5746 50  0000 L CNN
 F 1 "4.7k" H 4670 5655 50  0000 L CNN
-F 2 "" V 4530 5700 50  0001 C CNN
+F 2 "Resistor_SMD:R_0603_1608Metric" V 4530 5700 50  0001 C CNN
 F 3 "~" H 4600 5700 50  0001 C CNN
+F 4 "https://datasheet.lcsc.com/szlcsc/Uniroyal-Elec-0603WAF4701T5E_C23162.pdf" H 4600 5700 50  0001 C CNN "JLPCB Datasheet"
+F 5 "0603WAF4701T5E " H 4600 5700 50  0001 C CNN "JLPCB Part"
 	1    4600 5700
 	0    1    1    0
