File: Loader.sch (KiCad schematic (older format))
At the start: 51 parts, among them J1 USB_B_Micro, J2 I2C, J3 USB, J4 SPI, J5 LOADER_CON, J6 68KT_CON, J7 SPARE, J8 SPARE, J9 SPARE, SW1 SW_LOADER_RESET, U3 FT232RL, U4 ATmega2560-16AU, Y1 16MHz

Commit message: updates
Parts:
- removed C4: 10nF, symbol Device:CP
- removed C7: 4.7uF, symbol Device:CP
- removed D1: PWR_GREEN, symbol Device:LED
- removed FB1: Ferrite_Bead, symbol Device:Ferrite_Bead
- removed J1: USB_B_Micro, symbol Connector:USB_B_Micro
- removed J2: I2C, symbol Connector_Generic:Conn_01x03
- removed J3: USB, symbol Connector_Generic:Conn_01x04
- removed J4: SPI, symbol Connector_Generic:Conn_01x04
- removed J5: LOADER_CON, symbol Connector_Generic:Conn_01x03
- removed J6: 68KT_CON, symbol Connector_Generic:Conn_01x03
- removed R81: 82, symbol Device:R
Connections:
- no-connect marks 19 -> 18
Other:
- note added: "https://datasheet.lcsc.com/szlcsc/Future-Designs-FT232RL-REEL_C8690.pdf\nhttps://datasheet.lcsc.com/szlcsc/Microchip-Tech-ATMEGA2560-16AU_C22460.pdf"
- note removed: "https://www.amazon.co.uk/YOUMILE-Connector-Adapter-2-54mm-Converter-Microusb/dp/B07TVHR9LF\nhttps://datasheet.lcsc.com/szlcsc/Future-Designs-FT232RL-REEL_C8690.pdf\nhttps://datasheet.lcsc.com/szlcsc/Microchip-Tech-ATMEGA2560-16AU_C22460.pdf"
- moved on the sheet: C10, C11, C12, C3, C5, C6, D10, D11, D12, D2, D3, D4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

Commit message: updates
Parts:
- added D? (x2): LED7_RED, symbol Device:LED
- added SW?: SW_LOADER_RESET, symbol Switch:SW_Push
- added U? (x7): 74HCT04, symbol 74xx:74HCT04
Connections:
- net GND: now also D?.1 (K)
- net ~HALT: now also U?.1
- net ~RESET: now also U?.3
- new net: D?.2 (A), U?.2
- new net: D?.2 (A), U?.4
Changed lines of the file:
@@
 Wire Wire Line
 	3000 4800 3000 4600
+$Comp
+L Switch:SW_Push SW?
+U 1 1 5FE25891
+P 7500 2600
+F 0 "SW?" H 7500 2885 50  0000 C CNN
+F 1 "SW_LOADER_RESET" H 7500 2794 50  0000 C CNN
+F 2 "" H 7500 2800 50  0001 C CNN
+F 3 "~" H 7500 2800 50  0001 C CNN
+	1    7500 2600
+	1    0    0    -1
+$EndComp
+$Comp
+L 74xx:74HCT04 U?
+U 1 1 5FE3620D
+P 8250 3700
+F 0 "U?" H 8250 4017 50  0000 C CNN
+F 1 "74HCT04" H 8250 3926 50  0000 C CNN
+F 2 "" H 8250 3700 50  0001 C CNN
+F 3 "https://assets.nexperia.com/documents/data-sheet/74HC_HCT04.pdf" H 8250 3700 50  0001 C CNN
+	1    8250 3700
+	1    0    0    -1
+$EndComp
+$Comp
+L 74xx:74HCT04 U?
+U 2 1 5FE379C6
+P 7800 5200
+F 0 "U?" H 7800 5517 50  0000 C CNN
+F 1 "74HCT04" H 7800 5426 50  0000 C CNN
+F 2 "" H 7800 5200 50  0001 C CNN
+F 3 "https://assets.nexperia.com/documents/data-sheet/74HC_HCT04.pdf" H 7800 5200 50  0001 C CNN
+	2    7800 5200
+	1    0    0    -1
+$EndComp
+$Comp
+L 74xx:74HCT04 U?
+U 3 1 5FE3B3F5
+P 12250 2950
+F 0 "U?" H 12250 3267 50  0000 C CNN
+F 1 "74HCT04" H 12250 3176 50  0000 C CNN
+F 2 "" H 12250 2950 50  0001 C CNN
+F 3 "https://assets.nexperia.com/documents/data-sheet/74HC_HCT04.pdf" H 12250 2950 50  0001 C CNN
+	3    12250 2950
+	1    0    0    -1
+$EndComp
+$Comp
+L 74xx:74HCT04 U?
+U 4 1 5FE3D85A
+P 12350 3550
+F 0 "U?" H 12350 3867 50  0000 C CNN
+F 1 "74HCT04" H 12350 3776 50  0000 C CNN
+F 2 "" H 12350 3550 50  0001 C CNN
+F 3 "https://assets.nexperia.com/documents/data-sheet/74HC_HCT04.pdf" H 12350 3550 50  0001 C CNN
+	4    12350 3550
+	1    0    0    -1
+$EndComp
+$Comp
+L 74xx:74HCT04 U?
+U 5 1 5FE3EF29
+P 13150 2850
+F 0 "U?" H 13150 3167 50  0000 C CNN
+F 1 "74HCT04" H 13150 3076 50  0000 C CNN
+F 2 "" H 13150 2850 50  0001 C CNN
+F 3 "https://assets.nexperia.com/documents/data-sheet/74HC_HCT04.pdf" H 13150 2850 50  0001 C CNN
+	5    13150 2850
+	1    0    0    -1
+$EndComp
+$Comp
+L 74xx:74HCT04 U?
+U 6 1 5FE404BC
+P 13250 3550
+F 0 "U?" H 13250 3867 50  0000 C CNN
+F 1 "74HCT04" H 13250 3776 50  0000 C CNN
+F 2 "" H 13250 3550 50  0001 C CNN
+F 3 "https://assets.nexperia.com/documents/data-sheet/74HC_HCT04.pdf" H 13250 3550 50  0001 C CNN
+	6    13250 3550
+	1    0    0    -1
+$EndComp
+$Comp
+L 74xx:74HCT04 U?
+U 7 1 5FE41EF5
+P 14100 3650
+F 0 "U?" H 14330 3696 50  0000 L CNN
+F 1 "74HCT04" H 14330 3605 50  0000 L CNN
+F 2 "" H 14100 3650 50  0001 C CNN
+F 3 "https://assets.nexperia.com/documents/data-sheet/74HC_HCT04.pdf" H 14100 3650 50  0001 C CNN
+	7    14100 3650
+	1    0    0    -1
+$EndComp
+$Comp
+L Device:LED D?
+U 1 1 5FE5C9AF
+P 8550 3850
+AR Path="/5F9D5E69/5FE5C9AF" Ref="D?"  Part="1"
+AR Path="/5F9DA3F8/5FE5C9AF" Ref="D?"  Part="1"
+F 0 "D?" V 8589 3732 50  0000 R CNN
+F 1 "LED7_RED" V 8498 3732 50  0000 R CNN
+F 2 "" H 8550 3850 50  0001 C CNN
+F 3 "~" H 8550 3850 50  0001 C CNN
+	1    8550 3850
+	0    -1   -1   0
+$EndComp
+$Comp
+L power:GND #PWR?
+U 1 1 5FE5DBCA
+P 8500 4400
+F 0 "#PWR?" H 8500 4150 50  0001 C CNN
+F 1 "GND" H 8505 4227 50  0000 C CNN
+F 2 "" H 8500 4400 50  0001 C CNN
+F 3 "" H 8500 4400 50  0001 C CNN
+	1    8500 4400
+	1    0    0    -1
+$EndComp
+$Comp
+L Device:LED D?
+U 1 1 5FE71803
+P 8100 5350
+AR Path="/5F9D5E69/5FE71803" Ref="D?"  Part="1"
+AR Path="/5F9DA3F8/5FE71803" Ref="D?"  Part="1"
+F 0 "D?" V 8139 5232 50  0000 R CNN
+F 1 "LED7_RED" V 8048 5232 50  0000 R CNN
+F 2 "" H 8100 5350 50  0001 C CNN
+F 3 "~" H 8100 5350 50  0001 C CNN
+	1    8100 5350
+	0    -1   -1   0
+$EndComp
+$Comp
+L power:GND #PWR?
+U 1 1 5FE71809
+P 8100 5500
+F 0 "#PWR?" H 8100 5250 50  0001 C CNN
+F 1 "GND" H 8105 5327 50  0000 C CNN
+F 2 "" H 8100 5500 50  0001 C CNN
+F 3 "" H 8100 5500 50  0001 C CNN
+	1    8100 5500
+	1    0    0    -1
+$EndComp
+Text GLabel 7950 3700 0    50   Input ~ 0
+~HALT
+Text GLabel 7500 5200 0    50   Input ~ 0
+~RESET
 $EndSCHEMATC

Commit message: updates
Parts:
- removed C10, C11: 22nF, symbol Device:C
- removed D? (x2): LED7_RED, symbol Device:LED
- removed J7: SPARE, symbol Connector:Conn_01x08_Male
- removed J8: SPARE, symbol Connector:Conn_01x05_Male
- removed J9: SPARE, symbol Connector:Conn_01x04_Male
- removed SW?: SW_LOADER_RESET, symbol Switch:SW_Push
- removed U? (x7): 74HCT04, symbol 74xx:74HCT04
- added C13, C14: 22nF, symbol Device:C
- added TP10: Test Lader Reset, TestPoint:TestPoint_Pad_D1.0mm, symbol Connector:TestPoint
- added TP5: Test MISO, TestPoint:TestPoint_Pad_D1.0mm, symbol Connector:TestPoint
- added TP6: Test MOSI, TestPoint:TestPoint_Pad_D1.0mm, symbol Connector:TestPoint
- added TP7: Test SCK, TestPoint:TestPoint_Pad_D1.0mm, symbol Connector:TestPoint
- added TP8: Test SDA, TestPoint:TestPoint_Pad_D1.0mm, symbol Connector:TestPoint
- added TP9: Test SCL, TestPoint:TestPoint_Pad_D1.0mm, symbol Connector:TestPoint
- C12: renamed from C3; footprint (none) -> Capacitor_SMD:C_0603_1608Metric; JLPCB Datasheet (none) -> https://datasheet.lcsc.com/szlcsc/YAGEO-CC0603KRX7R9BB104_C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; JLPCB Part (none) -> CC0603KRX7R9BB104
- C15: renamed from C12; footprint (none) -> Capacitor_SMD:C_0603_1608Metric; JLPCB Datasheet (none) -> https://datasheet.lcsc.com/szlcsc/YAGEO-CC0603KRX7R9BB104_C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; JLPCB Part (none) -> CC0603KRX7R9BB104
- C16: renamed from C5; footprint (none) -> Capacitor_SMD:C_0603_1608Metric; JLPCB Datasheet (none) -> https://datasheet.lcsc.com/szlcsc/YAGEO-CC0603KRX7R9BB104_C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; JLPCB Part (none) -> CC0603KRX7R9BB104
- C17: renamed from C6; footprint (none) -> Capacitor_SMD:C_0603_1608Metric; JLPCB Datasheet (none) -> https://datasheet.lcsc.com/szlcsc/YAGEO-CC0603KRX7R9BB104_C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; JLPCB Part (none) -> CC0603KRX7R9BB104
- C18: renamed from C8; footprint (none) -> Capacitor_SMD:C_0603_1608Metric; JLPCB Datasheet (none) -> https://datasheet.lcsc.com/szlcsc/YAGEO-CC0603KRX7R9BB104_C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; JLPCB Part (none) -> CC0603KRX7R9BB104
- C19: renamed from C9; footprint (none) -> Capacitor_SMD:C_0603_1608Metric; JLPCB Datasheet (none) -> https://datasheet.lcsc.com/szlcsc/YAGEO-CC0603KRX7R9BB104_C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; JLPCB Part (none) -> CC0603KRX7R9BB104
- D10, D4: footprint (none) -> LED_SMD:LED_0603_1608Metric; JLPCB Datasheet (none) -> https://datasheet.lcsc.com/szlcsc/Hubei-KENTO-Elec-KT-0603R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; JLPCB Part (none) -> KT-0603R
- D11: renamed from D12; footprint (none) -> LED_SMD:LED_0603_1608Metric; JLPCB Datasheet (none) -> https://datasheet.lcsc.com/szlcsc/Hubei-KENTO-Elec-KT-0603R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; JLPCB Part (none) -> KT-0603R
- D2: value TX_GREEN -> TX_LED_GREEN; footprint (none) -> LED_SMD:LED_0603_1608Metric; JLPCB Datasheet (none) -> https://datasheet.lcsc.com/szlcsc/Everlight-Elec-19-217-GHC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; JLPCB Part (none) -> 19-217/GHC-YR1S2/3T
- D3: value RX_GREEN -> RX_LED_GREEN; footprint (none) -> LED_SMD:LED_0603_1608Metric; JLPCB Datasheet (none) -> https://datasheet.lcsc.com/szlcsc/Everlight-Elec-19-217-GHC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; JLPCB Part (none) -> 19-217/GHC-YR1S2/3T
- D5: renamed from D7; footprint (none) -> LED_SMD:LED_0603_1608Metric; JLPCB Datasheet (none) -> https://datasheet.lcsc.com/szlcsc/Hubei-KENTO-Elec-KT-0603R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; JLPCB Part (none) -> KT-0603R
- D6: renamed from D9; footprint (none) -> LED_SMD:LED_0603_1608Metric; JLPCB Datasheet (none) -> https://datasheet.lcsc.com/szlcsc/Hubei-KENTO-Elec-KT-0603R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; JLPCB Part (none) -> KT-0603R
- D7: renamed from D11; footprint (none) -> LED_SMD:LED_0603_1608Metric; JLPCB Datasheet (none) -> https://datasheet.lcsc.com/szlcsc/Hubei-KENTO-Elec-KT-0603R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; JLPCB Part (none) -> KT-0603R
- D8: renamed from D5; footprint (none) -> LED_SMD:LED_0603_1608Metric; JLPCB Datasheet (none) -> https://datasheet.lcsc.com/szlcsc/Hubei-KENTO-Elec-KT-0603R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; JLPCB Part (none) -> KT-0603R
- D9: renamed from D8; footprint (none) -> LED_SMD:LED_0603_1608Metric; JLPCB Datasheet (none) -> https://datasheet.lcsc.com/szlcsc/Hubei-KENTO-Elec-KT-0603R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; JLPCB Part (none) -> KT-0603R
- R11: renamed from R82; footprint (none) -> Resistor_SMD:R_0603_1608Metric; JLPCB Datasheet (none) -> https://datasheet.lcsc.com/szlcsc/Uniroyal-Elec-0603WAF820J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; JLPCB Part (none) -> 0603WAF820JT5E
- R12: renamed from R83; footprint (none) -> Resistor_SMD:R_0603_1608Metric; JLPCB Datasheet (none) -> https://datasheet.lcsc.com/szlcsc/Uniroyal-Elec-0603WAF820J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; JLPCB Part (none) -> 0603WAF820JT5E
- R14: renamed from R86; footprint (none) -> Resistor_SMD:R_0603_1608Metric; JLPCB Datasheet (none) -> https://datasheet.lcsc.com/szlcsc/Uniroyal-Elec-0603WAF1500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; JLPCB Part (none) -> 0603WAF1500T5E
- R16: renamed from R88; footprint (none) -> Resistor_SMD:R_0603_1608Metric; JLPCB Datasheet (none) -> https://datasheet.lcsc.com/szlcsc/Uniroyal-Elec-0603WAF1500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; JLPCB Part (none) -> 0603WAF1500T5E
- R17: renamed from R91; footprint (none) -> Resistor_SMD:R_0603_1608Metric; JLPCB Datasheet (none) -> https://datasheet.lcsc.com/szlcsc/Uniroyal-Elec-0603WAF1500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; JLPCB Part (none) -> 0603WAF1500T5E
- R18: renamed from R93; footprint (none) -> Resistor_SMD:R_0603_1608Metric; JLPCB Datasheet (none) -> https://datasheet.lcsc.com/szlcsc/Uniroyal-Elec-0603WAF1500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; JLPCB Part (none) -> 0603WAF1500T5E
- R19: renamed from R87; footprint (none) -> Resistor_SMD:R_0603_1608Metric; JLPCB Datasheet (none) -> https://datasheet.lcsc.com/szlcsc/Uniroyal-Elec-0603WAF1500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; JLPCB Part (none) -> 0603WAF1500T5E
- R20: renamed from R89; footprint (none) -> Resistor_SMD:R_0603_1608Metric; JLPCB Datasheet (none) -> https://datasheet.lcsc.com/szlcsc/Uniroyal-Elec-0603WAF1500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; JLPCB Part (none) -> 0603WAF1500T5E
- R21: renamed from R92; footprint (none) -> Resistor_SMD:R_0603_1608Metric; JLPCB Datasheet (none) -> https://datasheet.lcsc.com/szlcsc/Uniroyal-Elec-0603WAF1500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; JLPCB Part (none) -> 0603WAF1500T5E
- R22: renamed from R94; footprint (none) -> Resistor_SMD:R_0603_1608Metric; JLPCB Datasheet (none) -> https://datasheet.lcsc.com/szlcsc/Uniroyal-Elec-0603WAF1500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; JLPCB Part (none) -> 0603WAF1500T5E
- Y1: value 16MHz -> 8Mhz; footprint (none) -> Crystal:Crystal_SMD_5032-4Pin_5.0x3.2mm; JLPCB Datasheet (none) -> https://datasheet.lcsc.com/szlcsc/1903061615_Yangxing-Tech-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; JLPCB Part (none) -> X50328MSB2GI
- renumbered D6 to D1, R95 to R10, R84 to R13, R85 to R15, R90 to R9, U3 to U8, U4 to U9
Connections:
- net GND: now also C13.1, C14.1
- net MISO: now also TP5.1
- net MOSI: now also TP6.1
- net SCK: now also TP7.1
- net SCL: now also TP9.1
- net SDA: now also TP8.1
- net XTAL1: now also C13.2
- net XTAL2: now also C14.2
- net ~LOADER_RESET: now also TP10.1
- no-connect marks 18 -> 35
Other:
- note added: "Design from FT232RL datasheet page 19 and 20 (Capacitor values from datasheet):\nhttps://datasheet.lcsc.com/szlcsc/Future-Designs-FT232RL-REEL_C8690.pdf\n19-217/GHC-YR1S2/3T LIGHT EMITTING DIODES (LED) GREEN 520~535NM 112~258MCD@20MA TOP VIEW 0603 ROHS Basic Part\n0603WAF820JT5E CHIP RESISTOR - SURFACE MOUNT 82OHMS ±1% 1/10W 0603 ROH\n\nvcc=5; i=20; vf=3.3; (vcc-vf)/(i/1000); (i/1000)*(vcc-vf) = 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"
- note added: "Pseudo IO Memory Map\n$200001 CONSOLERX (A1)\n$200002 CONSOLETX (A2)\n$200004 LED0 (A3)\n$200008 LED1 (A4)\n$200010 LED2 (A5)\n$200020 LED3 (A6)\n$200040 LED4 (A7)\n$200080 LED5 (A8)\n$200100 LED6 (A9)\n$200200 LED7 (A10)\n$200400 RTCRX (A11)\n$200800 RTCTX (A12)\n$201000 FUTURE (A13)\n$202000 FUTURE (A14)\n$204000 FUTURE (A15)\n$208000 FUTURE (A16)\n$210000 FUTURE (A17)\n$220000 FUTURE (A18)\n$2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"
- note added: "https://datasheet.lcsc.com/szlcsc/Future-Designs-FT232RL-REEL_C8690.pdf\nhttps://datasheet.lcsc.com/szlcsc/Microchip-Tech-ATMEGA2560-16AU_C22460.pdf\nhttps://www.mouser.co.uk/datasheet/2/268/Atmel-2549-8-bit-AVR-Microcontroller-ATmega640-128-1315286.pdf"
- note added: "https://www.mouser.co.uk/datasheet/2/268/Atmel-2549-8-bit-AVR-Microcontroller-ATmega640-128-1315286.pdf\npage 42\nFrequency Range [MHz] 8.0 - 16.0, Recommended Range for Capacitors C1 and C2 [pF] 12 - 22\nMaximum frequency when using ceramic oscillator is 10MHz\nUse 8Mhz:\nX50328MSB2GI SMD CRYSTAL RESONATORS 8MHZ ±10PPM SMD-5032_2P ROHS\ncl=20; c0=1.8+5; 2*(cl-c0) Cap: 26.4 uF\n"
- note removed: "https://datasheet.lcsc.com/szlcsc/Future-Designs-FT232RL-REEL_C8690.pdf\nhttps://datasheet.lcsc.com/szlcsc/Microchip-Tech-ATMEGA2560-16AU_C22460.pdf"

Commit message: updates
Parts:
- D1: footprint (none) -> Diode_SMD:D_SMA; JLPCB Datasheet (none) -> https://datasheet.lcsc.com/szlcsc/MDD-Jiangsu-Yutai-Elec-M7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; JLPCB Part (none) -> M7
- TP1: renamed from TP5; JLPCB Datasheet (none) -> N/A; JLPCB Part (none) -> N/A
- TP2: renamed from TP6; JLPCB Datasheet (none) -> N/A; JLPCB Part (none) -> N/A
- TP3: renamed from TP7; JLPCB Datasheet (none) -> N/A; JLPCB Part (none) -> N/A
- TP4: renamed from TP8; JLPCB Datasheet (none) -> N/A; JLPCB Part (none) -> N/A
- TP5: renamed from TP9; JLPCB Datasheet (none) -> N/A; JLPCB Part (none) -> N/A
- TP6: renamed from TP10; JLPCB Datasheet (none) -> N/A; JLPCB Part (none) -> N/A
- U8: JLPCB Datasheet (none) -> https://datasheet.lcsc.com/szlcsc/Future-Designs-FT232RL-RE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; JLPCB Part (none) -> FT232RL-REEL
- renumbered D7 to D10, D8 to D5, D5 to D6, D9 to D7, D6 to D8, D10 to D9, R19 to R15, R15 to R16, R16 to R17, R20 to R18, R17 to R19, R21 to R20, R18 to R21
Connections:
- net WR is gone; now on net UDS: U9.96 (PF1)
- net AS: now also U9.93 (PF4); no longer U9.92 (PF5)
- net LDS: now also U9.95 (PF2); no longer U9.94 (PF3)
- net UDS: no longer U9.95 (PF2)
- net ~DTACK: now also U9.94 (PF3); no longer U9.93 (PF4)
- net RD renamed RW
- no-connect marks 35 -> 36
Other:
- note added: "Pseudo IO Memory Map\n$200001 CONSOLERX (A1)\n$200002 CONSOLETX (A2)\n$200004 LED0 (A3)\n$200008 LED1 (A4)\n$200010 LED2 (A5)\n$200020 LED3 (A6)\n$200040 LED4 (A7)\n$200080 LED5 (A8)\n$200100 LED6 (A9)\n$200200 LED7 (A10)\n$200400 RTCRX (A11)\n$200800 RTCTX (A12)\n$201000 LINKRX (A13)\n$202000 LINKTX (A14)\n$204000 FUTURE (A15)\n$208000 FUTURE (A16)\n$210000 FUTURE (A17)\n$220000 FUTURE (A18)\n$2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"
- note added: "http://ww1.microchip.com/downloads/en/appnotes/atmel-2521-\navr-hardware-design-considerations_applicationnote_avr042.pdf (Page 6&7)"
- note added: "https://datasheet.lcsc.com/szlcsc/Microchip-Tech-ATMEGA2560-16AU_C22460.pdf\nhttps://www.mouser.co.uk/datasheet/2/268/Atmel-2549-8-bit-AVR-Microcontroller-\nATmega640-128-1315286.pdf"
- note added: "https://www.mouser.co.uk/datasheet/2/268/Atmel-2549-8-\nbit-AVR-Microcontroller-ATmega640-128-1315286.pdf (page 42)\nFrequency Range [MHz] 8.0 - 16.0\nRecommended Range for Capacitors C1 and C2 [pF] 12 - 22\nMaximum frequency when using ceramic oscillator is 10MHz\nUse 8Mhz: X50328MSB2GI SMD CRYSTAL RESONATORS 8MHZ ±10PPM SMD-5032_2P ROHS\ncl=20; c0=1.8+5; 2*(cl-c0) = 26.4 uF\n"
- note removed: "Pseudo IO Memory Map\n$200001 CONSOLERX (A1)\n$200002 CONSOLETX (A2)\n$200004 LED0 (A3)\n$200008 LED1 (A4)\n$200010 LED2 (A5)\n$200020 LED3 (A6)\n$200040 LED4 (A7)\n$200080 LED5 (A8)\n$200100 LED6 (A9)\n$200200 LED7 (A10)\n$200400 RTCRX (A11)\n$200800 RTCTX (A12)\n$201000 FUTURE (A13)\n$202000 FUTURE (A14)\n$204000 FUTURE (A15)\n$208000 FUTURE (A16)\n$210000 FUTURE (A17)\n$220000 FUTURE (A18)\n$2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"
- note removed: "https://datasheet.lcsc.com/szlcsc/Future-Designs-FT232RL-REEL_C8690.pdf\nhttps://datasheet.lcsc.com/szlcsc/Microchip-Tech-ATMEGA2560-16AU_C22460.pdf\nhttps://www.mouser.co.uk/datasheet/2/268/Atmel-2549-8-bit-AVR-Microcontroller-ATmega640-128-1315286.pdf"
- note removed: "https://www.mouser.co.uk/datasheet/2/268/Atmel-2549-8-bit-AVR-Microcontroller-ATmega640-128-1315286.pdf\npage 42\nFrequency Range [MHz] 8.0 - 16.0, Recommended Range for Capacitors C1 and C2 [pF] 12 - 22\nMaximum frequency when using ceramic oscillator is 10MHz\nUse 8Mhz:\nX50328MSB2GI SMD CRYSTAL RESONATORS 8MHZ ±10PPM SMD-5032_2P ROHS\ncl=20; c0=1.8+5; 2*(cl-c0) Cap: 26.4 uF\n"
- moved on the sheet: C12, C13, C14, C15, C16, C17, C18, C19, D1, D10, D11, D2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

Commit message: update
Parts:
- C13, C14: footprint (none) -> Capacitor_SMD:C_0603_1608Metric
- R10: footprint (none) -> Resistor_SMD:R_0603_1608Metric; JLPCB Datasheet (none) -> https://datasheet.lcsc.com/szlcsc/Uniroyal-Elec-0603WAF3300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; JLPCB Part (none) -> 0603WAF3300T5E
- R13, R16: footprint (none) -> Resistor_SMD:R_0603_1608Metric; JLPCB Datasheet (none) -> https://datasheet.lcsc.com/szlcsc/Uniroyal-Elec-0603WAF1002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; JLPCB Part (none) -> 0603WAF1002T5E
- R9: footprint (none) -> Resistor_SMD:R_0603_1608Metric; JLPCB Datasheet (none) -> https://datasheet.lcsc.com/szlcsc/Uniroyal-Elec-0603WAF4701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; JLPCB Part (none) -> 0603WAF4701T5E
- SW1: footprint (none) -> Button_Switch_SMD:SW_Push_1P1T_NO_6x6mm_H9.5mm; JLPCB Datasheet (none) -> https://datasheet.lcsc.com/szlcsc/2006230332_USAKRO-UK-B022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; JLPCB Part (none) -> UK-B0228-G5-160-JZ
Changed lines of the file:
@@
 F 0 "R16" H 7370 3796 50  0000 L CNN
 F 1 "10k" H 7370 3705 50  0000 L CNN
-F 2 "" V 7230 3750 50  0001 C CNN
+F 2 "Resistor_SMD:R_0603_1608Metric" V 7230 3750 50  0001 C CNN
 F 3 "~" H 7300 3750 50  0001 C CNN
+F 4 "https://datasheet.lcsc.com/szlcsc/Uniroyal-Elec-0603WAF1002T5E_C25804.pdf" H 7300 3750 50  0001 C CNN "JLPCB Datasheet"
+F 5 "0603WAF1002T5E" H 7300 3750 50  0001 C CNN "JLPCB Part"
 	1    7300 3750
 	1    0    0    -1
@@
 F 0 "R13" H 7020 3796 50  0000 L CNN
 F 1 "10k" H 7020 3705 50  0000 L CNN
-F 2 "" V 6880 3750 50  0001 C CNN
+F 2 "Resistor_SMD:R_0603_1608Metric" V 6880 3750 50  0001 C CNN
 F 3 "~" H 6950 3750 50  0001 C CNN
+F 4 "https://datasheet.lcsc.com/szlcsc/Uniroyal-Elec-0603WAF1002T5E_C25804.pdf" H 6950 3750 50  0001 C CNN "JLPCB Datasheet"
+F 5 "0603WAF1002T5E" H 6950 3750 50  0001 C CNN "JLPCB Part"
 	1    6950 3750
 	1    0    0    -1
@@
 F 0 "SW1" H 2350 1635 50  0000 C CNN
 F 1 "SW_LOADER_RESET" H 2350 1544 50  0000 C CNN
-F 2 "" H 2350 1550 50  0001 C CNN
+F 2 "Button_Switch_SMD:SW_Push_1P1T_NO_6x6mm_H9.5mm" H 2350 1550 50  0001 C CNN
 F 3 "~" H 2350 1550 50  0001 C CNN
+F 4 "https://datasheet.lcsc.com/szlcsc/2006230332_USAKRO-UK-B0228-G5-160-JZ_C620316.pdf" H 2350 1350 50  0001 C CNN "JLPCB Datasheet"
+F 5 "UK-B0228-G5-160-JZ " H 2350 1350 50  0001 C CNN "JLPCB Part"
 	1    2350 1350
 	1    0    0    -1
@@
 F 0 "R9" H 1720 1146 50  0000 L CNN
 F 1 "4.7k" H 1720 1055 50  0000 L CNN
-F 2 "" V 1580 1100 50  0001 C CNN
+F 2 "Resistor_SMD:R_0603_1608Metric" V 1580 1100 50  0001 C CNN
 F 3 "~" H 1650 1100 50  0001 C CNN
+F 4 "https://datasheet.lcsc.com/szlcsc/Uniroyal-Elec-0603WAF4701T5E_C23162.pdf" H 1650 1100 50  0001 C CNN "JLPCB Datasheet"
+F 5 "0603WAF4701T5E " H 1650 1100 50  0001 C CNN "JLPCB Part"
 	1    1650 1100
 	1    0    0    -1
@@
 F 0 "R10" H 2720 1646 50  0000 L CNN
 F 1 "330" H 2720 1555 50  0000 L CNN
-F 2 "" V 2580 1600 50  0001 C CNN
+F 2 "Resistor_SMD:R_0603_1608Metric" V 2580 1600 50  0001 C CNN
 F 3 "~" H 2650 1600 50  0001 C CNN
+F 4 "https://datasheet.lcsc.com/szlcsc/Uniroyal-Elec-0603WAF3300T5E_C23138.pdf" H 2650 1600 50  0001 C CNN "JLPCB Datasheet"
+F 5 "0603WAF3300T5E" H 2650 1600 50  0001 C CNN "JLPCB Part"
 	1    2650 1600
 	1    0    0    -1
@@
 F 0 "C13" V 1400 2350 50  0000 R CNN
 F 1 "22nF" V 1500 2350 50  0000 R CNN
-F 2 "" H 1488 2250 50  0001 C CNN
+F 2 "Capacitor_SMD:C_0603_1608Metric" H 1488 2250 50  0001 C CNN
 F 3 "~" H 1450 2400 50  0001 C CNN
 	1    1450 2400
@@
 F 0 "C14" V 1400 3050 50  0000 R CNN
 F 1 "22nF" V 1500 3050 50  0000 R CNN
-F 2 "" H 1488 2950 50  0001 C CNN
+F 2 "Capacitor_SMD:C_0603_1608Metric" H 1488 2950 50  0001 C CNN
 F 3 "~" H 1450 3100 50  0001 C CNN
 	1    1450 3100
