File: Power.sch (KiCad schematic (older format))
At the start: 13 parts, among them U13 SRV05-4, U14 AMS1117-3.3

Commit message: updates
Parts:
- removed TP13: Test 3V, TestPoint:TestPoint_Pad_D1.0mm, symbol Connector:TestPoint
- added TP7: Test USB_VBUS, TestPoint:TestPoint_Pad_D1.0mm, symbol Connector:TestPoint
- added TP8: Test USB_D+, TestPoint:TestPoint_Pad_D1.0mm, symbol Connector:TestPoint
- added TP9: Test USB_D-, TestPoint:TestPoint_Pad_D1.0mm, symbol Connector:TestPoint
- TP10: renamed from TP11; JLPCB Datasheet (none) -> N/A; JLPCB Part (none) -> N/A
- TP11: renamed from TP12; JLPCB Datasheet (none) -> N/A; JLPCB Part (none) -> N/A
- U15: renamed from U13; JLPCB Datasheet (none) -> https://datasheet.lcsc.com/szlcsc/ProTek-Devices-SRV05-4-P-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; JLPCB Part (none) -> SRV05-4-P-T7
- renumbered R30 to R42, U14 to U16
Connections:
- net USB_D+: now also TP8.1
- net USB_D-: now also TP9.1
- net USB_VBUS: now also TP7.1
Other:
- note added: "Power: aprox 100mA\n\nFT232RL: 500mW @5.25V = 500/5.25 = 15mA\nATmega2560-16AU: 14mA\n10*LED=?\nIS62WV51216BLL: 35mA\n\n68000: 25mA\nGlue:\nLED:\n\n"
- note removed: "Power: aprox 100mA\n\nFT232RL: 500mW @5.25V = 500/5.25 = 15mA\nATmega2560-16AU: 14mA\n10*LED=?\nIS62WV51216BLL: 35mA\n40 * 2N7002 N-Channel Mosfets=?\n68000: 25mA\nGlue:\nLED:\n\n"
- moved on the sheet: TP10, TP11
Changed lines of the file:
@@
 AR Path="/5FA733C0" Ref="U?"  Part="1"
 AR Path="/60206568/5FA733C0" Ref="U?"  Part="1"
-AR Path="/5FA1AEF3/5FA733C0" Ref="U14"  Part="1"
-F 0 "U14" H 8350 1842 50  0000 C CNN
+AR Path="/5FA1AEF3/5FA733C0" Ref="U16"  Part="1"
+F 0 "U16" H 8350 1842 50  0000 C CNN
 F 1 "AMS1117-3.3" H 8350 1751 50  0000 C CNN
 F 2 "Package_TO_SOT_SMD:SOT-223-3_TabPin2" H 8350 1800 50  0001 C CNN
@@
 AR Path="/60206568/5FA733C6" Ref="#PWR?"  Part="1"
 AR Path="/5FA733C6" Ref="#PWR?"  Part="1"
-AR Path="/5FA1AEF3/5FA733C6" Ref="#PWR0113"  Part="1"
-F 0 "#PWR0113" H 7950 1350 50  0001 C CNN
+AR Path="/5FA1AEF3/5FA733C6" Ref="#PWR0121"  Part="1"
+F 0 "#PWR0121" H 7950 1350 50  0001 C CNN
 F 1 "+5V" H 7965 1673 50  0000 C CNN
 F 2 "" H 7950 1500 50  0001 C CNN
@@
 AR Path="/60206568/5FA733CC" Ref="#PWR?"  Part="1"
 AR Path="/5FA733CC" Ref="#PWR?"  Part="1"
-AR Path="/5FA1AEF3/5FA733CC" Ref="#PWR0116"  Part="1"
-F 0 "#PWR0116" H 8350 1750 50  0001 C CNN
+AR Path="/5FA1AEF3/5FA733CC" Ref="#PWR0123"  Part="1"
+F 0 "#PWR0123" H 8350 1750 50  0001 C CNN
 F 1 "GND" H 8355 1827 50  0000 C CNN
 F 2 "" H 8350 2000 50  0001 C CNN
@@
 AR Path="/60206568/5FA733D2" Ref="#PWR?"  Part="1"
 AR Path="/5FA733D2" Ref="#PWR?"  Part="1"
-AR Path="/5FA1AEF3/5FA733D2" Ref="#PWR0117"  Part="1"
-F 0 "#PWR0117" H 8750 1350 50  0001 C CNN
+AR Path="/5FA1AEF3/5FA733D2" Ref="#PWR0124"  Part="1"
+F 0 "#PWR0124" H 8750 1350 50  0001 C CNN
 F 1 "+3.3V" H 8765 1673 50  0000 C CNN
 F 2 "" H 8750 1500 50  0001 C CNN
@@
 AR Path="/60206568/5FA733DE" Ref="#PWR?"  Part="1"
 AR Path="/5FA733DE" Ref="#PWR?"  Part="1"
-AR Path="/5FA1AEF3/5FA733DE" Ref="#PWR0118"  Part="1"
-F 0 "#PWR0118" H 8750 1750 50  0001 C CNN
+AR Path="/5FA1AEF3/5FA733DE" Ref="#PWR0125"  Part="1"
+F 0 "#PWR0125" H 8750 1750 50  0001 C CNN
 F 1 "GND" H 8755 1827 50  0000 C CNN
 F 2 "" H 8750 2000 50  0001 C CNN
@@
 AR Path="/60206568/5FA733E4" Ref="#PWR?"  Part="1"
 AR Path="/5FA733E4" Ref="#PWR?"  Part="1"
-AR Path="/5FA1AEF3/5FA733E4" Ref="#PWR0114"  Part="1"
-F 0 "#PWR0114" H 7950 1750 50  0001 C CNN
+AR Path="/5FA1AEF3/5FA733E4" Ref="#PWR0122"  Part="1"
+F 0 "#PWR0122" H 7950 1750 50  0001 C CNN
 F 1 "GND" H 7955 1827 50  0000 C CNN
 F 2 "" H 7950 2000 50  0001 C CNN
@@
 AR Path="/5F9DA3F8/5FA733F9" Ref="#PWR?"  Part="1"
 AR Path="/5FA733F9" Ref="#PWR?"  Part="1"
-AR Path="/5FA1AEF3/5FA733F9" Ref="#PWR0110"  Part="1"
-F 0 "#PWR0110" H 3750 5300 50  0001 C CNN
+AR Path="/5FA1AEF3/5FA733F9" Ref="#PWR0120"  Part="1"
+F 0 "#PWR0120" H 3750 5300 50  0001 C CNN
 F 1 "GND" H 3755 5377 50  0000 C CNN
 F 2 "" H 3750 5550 50  0001 C CNN
@@
 AR Path="/5F9DA3F8/5FA7340B" Ref="#PWR?"  Part="1"
 AR Path="/5FA7340B" Ref="#PWR?"  Part="1"
-AR Path="/5FA1AEF3/5FA7340B" Ref="#PWR0109"  Part="1"
-F 0 "#PWR0109" H 3750 4400 50  0001 C CNN
+AR Path="/5FA1AEF3/5FA7340B" Ref="#PWR0119"  Part="1"
+F 0 "#PWR0119" H 3750 4400 50  0001 C CNN
 F 1 "+5V" H 3765 4723 50  0000 C CNN
 F 2 "" H 3750 4550 50  0001 C CNN
@@
 AR Path="/5F9DA3F8/5FA73417" Ref="R?"  Part="1"
 AR Path="/5FA73417" Ref="R?"  Part="1"
-AR Path="/5FA1AEF3/5FA73417" Ref="R30"  Part="1"
-F 0 "R30" H 3820 4946 50  0000 L CNN
+AR Path="/5FA1AEF3/5FA73417" Ref="R42"  Part="1"
+F 0 "R42" H 3820 4946 50  0000 L CNN
 F 1 "82" H 3820 4855 50  0000 L CNN
 F 2 "Resistor_SMD:R_0603_1608Metric" V 3680 4900 50  0001 C CNN
@@
 P 3000 1650
 AR Path="/5FA73442" Ref="U?"  Part="1"
-AR Path="/5FA1AEF3/5FA73442" Ref="U13"  Part="1"
-F 0 "U13" H 3150 2100 50  0000 C CNN
+AR Path="/5FA1AEF3/5FA73442" Ref="U15"  Part="1"
+F 0 "U15" H 3150 2100 50  0000 C CNN
 F 1 "SRV05-4" H 3250 2200 50  0000 C CNN
 F 2 "Package_TO_SOT_SMD:SOT-23-6" H 3700 1200 50  0001 C CNN
 F 3 "http://www.onsemi.com/pub/Collateral/SRV05-4-D.PDF" H 3000 1650 50  0001 C CNN
+F 4 "https://datasheet.lcsc.com/szlcsc/ProTek-Devices-SRV05-4-P-T7_C85364.pdf" H 3000 1650 50  0001 C CNN "JLPCB Datasheet"
+F 5 "SRV05-4-P-T7" H 3000 1650 50  0001 C CNN "JLPCB Part"
 	1    3000 1650
 	1    0    0    -1
@@
 	2750 5450 3250 5450
 Text Notes 8850 6450 0    50   ~ 0
-Power: aprox 100mA\n\nFT232RL:  500mW @5.25V = 500/5.25 = 15mA\nATmega2560-16AU: 14mA\n10*LED=?\nIS62WV51216BLL: 35mA\n40 * 2N7002 N-Channel Mosfets=?\n68000: 25mA\nGlue:\nLED:\n\n
-$Comp
-L Connector:TestPoint TP?
-U 1 1 5FA2FDE9
-P 7950 5950
-AR Path="/5F9DA3F8/5FA2FDE9" Ref="TP?"  Part="1"
-AR Path="/5FA1AEF3/5FA2FDE9" Ref="TP13"  Part="1"
-F 0 "TP13" H 8008 6068 50  0000 L CNN
-F 1 "Test 3V" H 8008 5977 50  0000 L CNN
-F 2 "TestPoint:TestPoint_Pad_D1.0mm" H 8150 5950 50  0001 C CNN
-F 3 "~" H 8150 5950 50  0001 C CNN
-	1    7950 5950
-	1    0    0    -1
-$EndComp
+Power: aprox 100mA\n\nFT232RL:  500mW @5.25V = 500/5.25 = 15mA\nATmega2560-16AU: 14mA\n10*LED=?\nIS62WV51216BLL: 35mA\n\n68000: 25mA\nGlue:\nLED:\n\n
 $Comp
 L Connector:TestPoint TP?
 U 1 1 5FA31527
-P 6750 5950
+P 9300 4300
 AR Path="/5F9DA3F8/5FA31527" Ref="TP?"  Part="1"
-AR Path="/5FA1AEF3/5FA31527" Ref="TP11"  Part="1"
-F 0 "TP11" H 6692 5976 50  0000 R CNN
-F 1 "Test 5V" H 6692 6067 50  0000 R CNN
-F 2 "TestPoint:TestPoint_Pad_D1.0mm" H 6950 5950 50  0001 C CNN
-F 3 "~" H 6950 5950 50  0001 C CNN
-	1    6750 5950
+AR Path="/5FA1AEF3/5FA31527" Ref="TP10"  Part="1"
+F 0 "TP10" H 9242 4326 50  0000 R CNN
+F 1 "Test 5V" H 9242 4417 50  0000 R CNN
+F 2 "TestPoint:TestPoint_Pad_D1.0mm" H 9500 4300 50  0001 C CNN
+F 3 "~" H 9500 4300 50  0001 C CNN
+F 4 "N/A" H 9300 4300 50  0001 C CNN "JLPCB Datasheet"
+F 5 "N/A" H 9300 4300 50  0001 C CNN "JLPCB Part"
+	1    9300 4300
 	-1   0    0    1
-$EndComp
-$Comp
-L power:GND #PWR?
-U 1 1 5FA36943
-P 7950 5950
-AR Path="/5F9D5E69/5FA36943" Ref="#PWR?"  Part="1"
-AR Path="/5F9DA3F8/5FA36943" Ref="#PWR?"  Part="1"
-AR Path="/5FA36943" Ref="#PWR?"  Part="1"
-AR Path="/5FA1AEF3/5FA36943" Ref="#PWR0115"  Part="1"
-F 0 "#PWR0115" H 7950 5700 50  0001 C CNN
-F 1 "GND" H 7955 5777 50  0000 C CNN
-F 2 "" H 7950 5950 50  0001 C CNN
-F 3 "" H 7950 5950 50  0001 C CNN
-	1    7950 5950
-	1    0    0    -1
 $EndComp
 $Comp
 L power:+5V #PWR?
 U 1 1 5FA36E10
-P 6750 5950
+P 9300 4300
 AR Path="/5F9D5E69/5FA36E10" Ref="#PWR?"  Part="1"
 AR Path="/5F9DA3F8/5FA36E10" Ref="#PWR?"  Part="1"
 AR Path="/5FA36E10" Ref="#PWR?"  Part="1"
-AR Path="/5FA1AEF3/5FA36E10" Ref="#PWR0111"  Part="1"
-F 0 "#PWR0111" H 6750 5800 50  0001 C CNN
-F 1 "+5V" H 6765 6123 50  0000 C CNN
-F 2 "" H 6750 5950 50  0001 C CNN
-F 3 "" H 6750 5950 50  0001 C CNN
-	1    6750 5950
+AR Path="/5FA1AEF3/5FA36E10" Ref="#PWR0126"  Part="1"
+F 0 "#PWR0126" H 9300 4150 50  0001 C CNN
+F 1 "+5V" H 9315 4473 50  0000 C CNN
+F 2 "" H 9300 4300 50  0001 C CNN
+F 3 "" H 9300 4300 50  0001 C CNN
+	1    9300 4300
 	1    0    0    -1
 $EndComp
@@
 L power:+3.3V #PWR?
 U 1 1 5FA37490
-P 7350 5950
+P 9900 4300
 AR Path="/60206568/5FA37490" Ref="#PWR?"  Part="1"
 AR Path="/5FA37490" Ref="#PWR?"  Part="1"
-AR Path="/5FA1AEF3/5FA37490" Ref="#PWR0112"  Part="1"
-F 0 "#PWR0112" H 7350 5800 50  0001 C CNN
-F 1 "+3.3V" H 7365 6123 50  0000 C CNN
-F 2 "" H 7350 5950 50  0001 C CNN
-F 3 "" H 7350 5950 50  0001 C CNN
-	1    7350 5950
+AR Path="/5FA1AEF3/5FA37490" Ref="#PWR0127"  Part="1"
+F 0 "#PWR0127" H 9900 4150 50  0001 C CNN
+F 1 "+3.3V" H 9915 4473 50  0000 C CNN
+F 2 "" H 9900 4300 50  0001 C CNN
+F 3 "" H 9900 4300 50  0001 C CNN
+	1    9900 4300
 	1    0    0    -1
 $EndComp
@@
 L Connector:TestPoint TP?
 U 1 1 5FA44775
-P 7350 5950
+P 9900 4300
 AR Path="/5F9DA3F8/5FA44775" Ref="TP?"  Part="1"
-AR Path="/5FA1AEF3/5FA44775" Ref="TP12"  Part="1"
-F 0 "TP12" H 7292 5976 50  0000 R CNN
-F 1 "Test 3V" H 7292 6067 50  0000 R CNN
-F 2 "TestPoint:TestPoint_Pad_D1.0mm" H 7550 5950 50  0001 C CNN
-F 3 "~" H 7550 5950 50  0001 C CNN
-	1    7350 5950
+AR Path="/5FA1AEF3/5FA44775" Ref="TP11"  Part="1"
+F 0 "TP11" H 9842 4326 50  0000 R CNN
+F 1 "Test 3V" H 9842 4417 50  0000 R CNN
+F 2 "TestPoint:TestPoint_Pad_D1.0mm" H 10100 4300 50  0001 C CNN
+F 3 "~" H 10100 4300 50  0001 C CNN
+F 4 "N/A" H 9900 4300 50  0001 C CNN "JLPCB Datasheet"
+F 5 "N/A" H 9900 4300 50  0001 C CNN "JLPCB Part"
+	1    9900 4300
 	-1   0    0    1
 $EndComp
+Text GLabel 7900 4050 0    50   Input ~ 0
+USB_VBUS
+Text GLabel 7900 4300 0    50   BiDi ~ 0
+USB_D+
+Text GLabel 7900 4500 0    50   BiDi ~ 0
+USB_D-
+$Comp
+L Connector:TestPoint TP?
+U 1 1 605DC408
+P 7900 4300
+AR Path="/5F9DA3F8/605DC408" Ref="TP?"  Part="1"
+AR Path="/605DC408" Ref="TP?"  Part="1"
+AR Path="/5FA1AEF3/605DC408" Ref="TP8"  Part="1"
+F 0 "TP8" V 7854 4488 50  0000 L CNN
+F 1 "Test USB_D+" V 7945 4488 50  0000 L CNN
+F 2 "TestPoint:TestPoint_Pad_D1.0mm" H 8100 4300 50  0001 C CNN
+F 3 "~" H 8100 4300 50  0001 C CNN
+F 4 "N/A" H 7900 4300 50  0001 C CNN "JLPCB Datasheet"
+F 5 "N/A" H 7900 4300 50  0001 C CNN "JLPCB Part"
+	1    7900 4300
+	0    1    1    0
+$EndComp
+$Comp
+L Connector:TestPoint TP?
+U 1 1 605DC40E
+P 7900 4500
+AR Path="/5F9DA3F8/605DC40E" Ref="TP?"  Part="1"
+AR Path="/605DC40E" Ref="TP?"  Part="1"
+AR Path="/5FA1AEF3/605DC40E" Ref="TP9"  Part="1"
+F 0 "TP9" V 7854 4688 50  0000 L CNN
+F 1 "Test USB_D-" V 7945 4688 50  0000 L CNN
+F 2 "TestPoint:TestPoint_Pad_D1.0mm" H 8100 4500 50  0001 C CNN
+F 3 "~" H 8100 4500 50  0001 C CNN
+F 4 "N/A" H 7900 4500 50  0001 C CNN "JLPCB Datasheet"
+F 5 "N/A" H 7900 4500 50  0001 C CNN "JLPCB Part"
+	1    7900 4500
+	0    1    1    0
+$EndComp
+$Comp
+L Connector:TestPoint TP?
+U 1 1 605DC41A
+P 7900 4050
+AR Path="/5F9DA3F8/605DC41A" Ref="TP?"  Part="1"
+AR Path="/605DC41A" Ref="TP?"  Part="1"
+AR Path="/5FA1AEF3/605DC41A" Ref="TP7"  Part="1"
+F 0 "TP7" V 7854 4238 50  0000 L CNN
+F 1 "Test USB_VBUS" V 7945 4238 50  0000 L CNN
+F 2 "TestPoint:TestPoint_Pad_D1.0mm" H 8100 4050 50  0001 C CNN
+F 3 "~" H 8100 4050 50  0001 C CNN
+F 4 "N/A" H 7900 4050 50  0001 C CNN "JLPCB Datasheet"
+F 5 "N/A" H 7900 4050 50  0001 C CNN "JLPCB Part"
+	1    7900 4050
+	0    1    1    0
+$EndComp
 $EndSCHEMATC

Commit message: update
Parts:
- C25, C27: footprint (none) -> Capacitor_SMD:C_0603_1608Metric
Changed lines of the file:
@@
 F 0 "C25" H 2368 5096 50  0000 L CNN
 F 1 "10nF" H 2368 5005 50  0000 L CNN
-F 2 "" H 2288 4900 50  0001 C CNN
+F 2 "Capacitor_SMD:C_0603_1608Metric" H 2288 4900 50  0001 C CNN
 F 3 "~" H 2250 5050 50  0001 C CNN
 	1    2250 5050
@@
 F 0 "C27" H 3368 5096 50  0000 L CNN
 F 1 "4.7uF" H 3368 5005 50  0000 L CNN
-F 2 "" H 3288 4900 50  0001 C CNN
+F 2 "Capacitor_SMD:C_0603_1608Metric" H 3288 4900 50  0001 C CNN
 F 3 "~" H 3250 5050 50  0001 C CNN
 	1    3250 5050
